File: solarpump.kicad_pcb (KiCad board)
At the start: 2 copper layers, 116.5 x 66 mm, 87 parts, among them J10 MotorSens_M, J11 MotorPowr_M, J16 Disply_M, J17 TchScr_M, J18 2 pin header, J5 Soldered, J6 Soldered, J8 XLR3 Male PCB, J9 XLR3 Male PCB, Q1 IRLB8721PBF, Q2 2N3904, Q3 2N3904, Q4 IRLB8721PBF, Q5 IRLB8721PBF, Q6 2N3904, Q7 IRLB8721PBF, Q8 2N3904, SW1 Rotary_Encoder_Switch, U1 IR2104, U1_C1 0.1uF, U1_C2 10uF, U2 LTC2992, U3 LTC2992, U4 LM2576HVS-5

Commit message: Update for v3
Parts:
- removed +Bat1, -Bat1: Soldered, Connector_Wire:SolderWire-1.5sqmm_1x01_D1.7mm_OD3.9mm
- removed +Bat2, -Bat2: Soldered, Connector_Wire:SolderWire-0.5sqmm_1x01_D0.9mm_OD2.3mm
- removed C_MCU1, C_U1, C_U2: 1uF, Capacitor_THT:C_Disc_D5.0mm_W2.5mm_P5.00mm
- removed HS_Q1, HS_Q4, HS_Q5, HS_Q7: H/S, solarpump:Heatsink_14x9.5mm
- removed J10: MotorSens_M, Connector_PinHeader_1.27mm:PinHeader_1x06_P1.27mm_Vertical
- removed J11: MotorPowr_M, Connector_Phoenix_MC:PhoenixContact_MCV_1,5_2-G-3.5_1x02_P3.50mm_Vertical
- removed J16: Disply_M, Connector_PinHeader_1.27mm:PinHeader_1x07_P1.27mm_Vertical
- removed J17: TchScr_M, Connector_PinHeader_1.27mm:PinHeader_1x06_P1.27mm_Vertical
- removed J18: 2 pin header, Connector_PinHeader_1.27mm:PinHeader_1x02_P1.27mm_Vertical
- removed JP3: Disable Q5 (NC), Jumper:SolderJumper-2_P1.3mm_Bridged_Pad1.0x1.5mm
- removed U1_C1: 0.1uF, Capacitor_THT:C_Disc_D5.0mm_W2.5mm_P5.00mm
- removed U1_C2: 10uF, Capacitor_THT:C_Disc_D5.0mm_W2.5mm_P5.00mm
- added BZ1: Buzzer, solarpump:Buzzer_3V, B.Cu at (85.8, 31.1)
- added C1: 10uF, Capacitor_SMD:C_0805_2012Metric_Pad1.18x1.45mm_HandSolder, F.Cu at (147.9, 143.8)
- added C13: 1uF, Capacitor_SMD:C_0805_2012Metric_Pad1.18x1.45mm_HandSolder, F.Cu at (157.2, 142.4)
- added C14: 100nF, Capacitor_SMD:C_0805_2012Metric_Pad1.18x1.45mm_HandSolder, F.Cu at (59.7, 76.4)
- added C15: 100nF, Capacitor_SMD:C_0805_2012Metric_Pad1.18x1.45mm_HandSolder, F.Cu at (132.4, 137.5)
- added C16: 100nF, Capacitor_SMD:C_0805_2012Metric_Pad1.18x1.45mm_HandSolder, F.Cu at (59.7, 72.4)
- added C17: 10nF, 50V, Capacitor_SMD:C_0805_2012Metric_Pad1.18x1.45mm_HandSolder, F.Cu at (107.7, 90.2)
- added C18: 100nF, Capacitor_SMD:C_0805_2012Metric_Pad1.18x1.45mm_HandSolder, F.Cu at (77.7, 94.5)
- added C19: 100nF, Capacitor_SMD:C_0805_2012Metric_Pad1.18x1.45mm_HandSolder, F.Cu at (77.2, 91.2)
- added C2: 0.1uF, Capacitor_SMD:C_0805_2012Metric_Pad1.18x1.45mm_HandSolder, F.Cu at (147.9, 141.8)
- added C20: 22uF,25V, Capacitor_SMD:C_1210_3225Metric_Pad1.33x2.70mm_HandSolder, F.Cu at (100.2, 85.6)
- added C21: 100nF, Capacitor_SMD:C_0805_2012Metric_Pad1.18x1.45mm_HandSolder, F.Cu at (142.5, 106.2)
- added C22: 100nF, Capacitor_SMD:C_0805_2012Metric_Pad1.18x1.45mm_HandSolder, F.Cu at (136.3, 137.5)
- added C23: 100nF, Capacitor_SMD:C_0805_2012Metric_Pad1.18x1.45mm_HandSolder, F.Cu at (138.5, 106.2)
- added C24: 47uF, Capacitor_THT:CP_Radial_D6.3mm_P2.50mm, F.Cu at (87.5, 141.5)
- added C25: 4.7uF, Capacitor_SMD:C_0805_2012Metric_Pad1.18x1.45mm_HandSolder, F.Cu at (66.3, 111.1)
- added C26: 47uF, Capacitor_THT:CP_Radial_D6.3mm_P2.50mm, F.Cu at (107.7, 141.6)
- added C27: 47uF, Capacitor_THT:CP_Radial_D6.3mm_P2.50mm, F.Cu at (66.9, 133.1)
- added C28: 4.7uF, Capacitor_SMD:C_0805_2012Metric_Pad1.18x1.45mm_HandSolder, F.Cu at (106.1, 129.1)
- added C29: 4.7uF, Capacitor_SMD:C_0805_2012Metric_Pad1.18x1.45mm_HandSolder, F.Cu at (85.9, 128.6)
- added C30: 47uF, Capacitor_SMD:C_1206_3216Metric_Pad1.33x1.80mm_HandSolder, F.Cu at (88.5, 129.2)
- added C31: 100n, Capacitor_THT:C_Disc_D5.0mm_W2.5mm_P5.00mm, F.Cu at (73.2, 44.1)
- added C32: 100n, Capacitor_THT:C_Disc_D5.0mm_W2.5mm_P5.00mm, F.Cu at (167.7, 40.9)
- added C33: 100n, Capacitor_THT:C_Disc_D5.0mm_W2.5mm_P5.00mm, F.Cu at (162.6, 40.8)
- added C34: 100n, Capacitor_THT:C_Disc_D5.0mm_W2.5mm_P5.00mm, F.Cu at (172.8, 40.9)
- added C35: 2nF, 50V, Capacitor_SMD:C_0805_2012Metric_Pad1.18x1.45mm_HandSolder, F.Cu at (186.3, 67.5)
- added C36: 22uF,25V, Capacitor_SMD:C_1210_3225Metric_Pad1.33x2.70mm_HandSolder, F.Cu at (203.7, 90.5)
- added C37: 22uF,25V, Capacitor_SMD:C_1210_3225Metric_Pad1.33x2.70mm_HandSolder, F.Cu at (200.5, 105.3)
- added C38: 22uF,25V, Capacitor_SMD:C_1210_3225Metric_Pad1.33x2.70mm_HandSolder, F.Cu at (204.0, 105.2)
- added C39: 100nF, Capacitor_SMD:C_0805_2012Metric_Pad1.18x1.45mm_HandSolder, F.Cu at (175.1, 81.9)
- added C40: 100nF, Capacitor_SMD:C_0805_2012Metric_Pad1.18x1.45mm_HandSolder, F.Cu at (136.5, 130.9)
- added C41: 100nF, Capacitor_SMD:C_0805_2012Metric_Pad1.18x1.45mm_HandSolder, F.Cu at (179.1, 81.9)
- added C42: 100nF, Capacitor_SMD:C_0805_2012Metric_Pad1.18x1.45mm_HandSolder, F.Cu at (132.4, 130.9)
- added C43: 100nF, Capacitor_SMD:C_0805_2012Metric_Pad1.18x1.45mm_HandSolder, F.Cu at (196.2, 107.3)
- added C44: 100nF, Capacitor_SMD:C_0805_2012Metric_Pad1.18x1.45mm_HandSolder, F.Cu at (192.2, 107.3)
- added CP1: 220uF, 50V, Capacitor_THT:CP_Radial_D12.5mm_P5.00mm, F.Cu at (71.7, 56.9)
- added CP2: 470uF,25V, Capacitor_THT:C_Radial_D10.0mm_H16.0mm_P5.00mm, F.Cu at (94.1, 91.6)
- added CP3: 470uF, 50V, Capacitor_THT:C_Radial_D12.5mm_H25.0mm_P5.00mm, F.Cu at (62.4, 141.6)
- added CP4: 470uF, 25V, Capacitor_THT:C_Radial_D10.0mm_H20.0mm_P5.00mm, F.Cu at (61.7, 102.8)
- added CP5: 390uF, 10V, Capacitor_THT:C_Radial_D10.0mm_H12.5mm_P5.00mm, F.Cu at (114.2, 129.2)
- added CP6: 390uF, 10V, Capacitor_THT:C_Radial_D10.0mm_H12.5mm_P5.00mm, F.Cu at (85.6, 123.0)
- added CP7: 470uF,25V, Capacitor_THT:C_Radial_D10.0mm_H16.0mm_P5.00mm, F.Cu at (208.6, 116.7)
- added D1: S07G-M, Diode_SMD:D_SOD-123, F.Cu at (58.8, 63.9)
- added D10: B140-E3/5AT, Diode_SMD:D_SOD-123, F.Cu at (182.0, 61.1)
- added D11: S07G-M, Diode_SMD:D_SOD-123, F.Cu at (149.4, 67.3)
- added D12: S07G-M, Diode_SMD:D_SOD-123, F.Cu at (157.7, 67.2)
- added D5: S07G-M, Diode_SMD:D_SOD-123, F.Cu at (121.7, 137.0)
- added D9: B140-E3/5AT, Diode_SMD:D_SOD-123, F.Cu at (206.9, 66.2)
- added F1: Fuse 25A, Fuse:Fuseholder_Keystone_3555-2, F.Cu at (112.8, 54.5)
- added F2: Fuse 25A, Fuse:Fuseholder_Keystone_3555-2, F.Cu at (159.9, 111.0)
- added H6: MountingHole, MountingHole:MountingHole_4.3mm_M4, F.Cu at (180.0, 18.7)
- added H7: MountingHole, MountingHole:MountingHole_4.3mm_M4, F.Cu at (180.0, 44.2)
- added H8: MountingHole, MountingHole:MountingHole_4.3mm_M4, F.Cu at (59.6, 44.2)
- added HS1: Heatsink, MountingHole:MountingHole_2.2mm_M2_Pad_Via, F.Cu at (84.1, 111.8)
- added HS2: Heatsink, MountingHole:MountingHole_2.2mm_M2_Pad_Via, F.Cu at (106.9, 111.8)
- added HS3: Heatsink, MountingHole:MountingHole_2.2mm_M2_Pad_Via, F.Cu at (151.7, 111.8)
- added HS4: Heatsink, MountingHole:MountingHole_2.2mm_M2_Pad_Via, F.Cu at (84.1, 87.0)
- added HS5: Heatsink, MountingHole:MountingHole_2.2mm_M2_Pad_Via, F.Cu at (176.4, 54.3)
- added HS6: Heatsink, MountingHole:MountingHole_2.2mm_M2_Pad_Via, F.Cu at (218.2, 54.3)
- added HS7: Heatsink, MountingHole:MountingHole_2.2mm_M2_Pad_Via, F.Cu at (130.7, 67.3)
- added HS8: Heatsink, MountingHole:MountingHole_2.2mm_M2_Pad_Via, F.Cu at (218.2, 68.8)
- added J1: 8-way_Screw, TerminalBlock_Phoenix:TerminalBlock_Phoenix_MKDS-3-8-5.08_1x08_P5.08mm_Horizontal, F.Cu at (135.2, 57.4)
- added J2: UART_IO, Connector_PinHeader_2.00mm:PinHeader_1x03_P2.00mm_Vertical, F.Cu at (170.6, 130.7)
- added J3: AUX_POWER, Connector_PinHeader_2.00mm:PinHeader_1x04_P2.00mm_Vertical, F.Cu at (207.2, 130.0)
- added J4: USB_A, solarpump:USB_Receptacle_Type_A_GCT, F.Cu at (220.3, 133.3)
- added L3: 100uH, Inductor_SMD:L_10.4x10.4_H4.8, F.Cu at (98.0, 132.7)
- added L4: 100uH, Inductor_SMD:L_10.4x10.4_H4.8, F.Cu at (77.6, 132.7)
- added L5: 68uH, Inductor_THT:L_Toroid_Vertical_L35.1mm_W21.1mm_P18.50mm_Vishay_TJ6, F.Cu at (226.2, 92.4)
- added M2: Pico_Display_Pack, Package_DIP:DIP-40_W15.24mm_Socket, F.Cu at (97.1, 38.5)
- added NT1: NetTie_2, NetTie:NetTie-2_THT_Pad1.0mm, F.Cu at (128.0, 124.7)
- added Q10: Si2306BDS, Package_TO_SOT_SMD:SOT-23, F.Cu at (173.3, 70.9)
- added Q11: IRLB8721PBF, Package_TO_SOT_THT:TO-220-3_Vertical, F.Cu at (148.3, 71.7)
- added Q12: IRLB8721PBF, Package_TO_SOT_THT:TO-220-3_Vertical, F.Cu at (163.9, 71.6)
- added Q9: Si2306BDS, Package_TO_SOT_SMD:SOT-23, F.Cu at (135.5, 72.8)
- added R10: 0, Resistor_SMD:R_0805_2012Metric_Pad1.20x1.40mm_HandSolder, F.Cu at (127.5, 94.2)
- added R24: 10k, Resistor_SMD:R_0805_2012Metric_Pad1.20x1.40mm_HandSolder, F.Cu at (158.3, 26.7)
- added R27: 0, Resistor_SMD:R_0805_2012Metric_Pad1.20x1.40mm_HandSolder, F.Cu at (182.0, 66.3)
- added R3: 6.8k, Resistor_SMD:R_0805_2012Metric_Pad1.20x1.40mm_HandSolder, F.Cu at (116.7, 154.0)
- added R30: 33k, Resistor_SMD:R_0805_2012Metric_Pad1.20x1.40mm_HandSolder, F.Cu at (167.0, 112.1)
- added R31: 1k, Resistor_SMD:R_0805_2012Metric_Pad1.20x1.40mm_HandSolder, F.Cu at (171.0, 112.1)
- added R32: 10k, Resistor_SMD:R_0805_2012Metric_Pad1.20x1.40mm_HandSolder, F.Cu at (132.2, 72.9)
- added R33: 10k, Resistor_SMD:R_0805_2012Metric_Pad1.20x1.40mm_HandSolder, F.Cu at (176.2, 71.0)
- added R34: 10k, Resistor_SMD:R_0805_2012Metric_Pad1.20x1.40mm_HandSolder, F.Cu at (135.5, 69.8)
- added R35: 10k, Resistor_SMD:R_0805_2012Metric_Pad1.20x1.40mm_HandSolder, F.Cu at (173.5, 73.9)
- added R36: 100, Resistor_SMD:R_0805_2012Metric_Pad1.20x1.40mm_HandSolder, F.Cu at (135.5, 75.9)
- added R37: 100, Resistor_SMD:R_0805_2012Metric_Pad1.20x1.40mm_HandSolder, F.Cu at (169.6, 70.4)
- added R38: 10k, Resistor_SMD:R_0805_2012Metric_Pad1.20x1.40mm_HandSolder, F.Cu at (139.0, 75.0)
- added R39: 10k, Resistor_SMD:R_0805_2012Metric_Pad1.20x1.40mm_HandSolder, F.Cu at (169.6, 72.9)
- added R40: 22k, Resistor_SMD:R_0805_2012Metric_Pad1.20x1.40mm_HandSolder, F.Cu at (132.4, 134.2)
- added R41: 1k, Resistor_SMD:R_0805_2012Metric_Pad1.20x1.40mm_HandSolder, F.Cu at (136.5, 134.2)
- added RN1: R_Network03_10K, Resistor_THT:R_Array_SIP4, F.Cu at (161.0, 147.0)
- added SW2: Rotary Enc EC11E, Rotary_Encoder:RotaryEncoder_Alps_EC11E-Switch_Vertical_H20mm, F.Cu at (162.5, 28.4)
- added TH1: 10K_Thermistor_NTC, solarpump:SolderWire-0.15sqmm_1x02_P3.5mm_D0.5mm_OD1.5mm, F.Cu at (168.3, 145.3)
- added TH2: 10K_Thermistor_NTC, solarpump:SolderWire-0.15sqmm_1x02_P3.5mm_D0.5mm_OD1.5mm, F.Cu at (168.3, 142.1)
- added TH3: 10K_Thermistor_NTC, solarpump:SolderWire-0.15sqmm_1x02_P3.5mm_D0.5mm_OD1.5mm, F.Cu at (168.3, 138.8)
- added TP1: VTEST+, TestPoint:TestPoint_Pad_1.0x1.0mm, F.Cu at (144.3, 146.3)
- added TP2: VTEST-, TestPoint:TestPoint_Pad_1.0x1.0mm, F.Cu at (146.9, 146.3)
- added U10: L6398D, Package_SO:SOIC-8_3.9x4.9mm_P1.27mm, F.Cu at (192.4, 66.6)
- added U11: ACS758xCB, solarpump:Allegro_CB_PFF, F.Cu at (179.0, 84.4)
- added U12: ACS758xCB, solarpump:Allegro_CB_PFF, F.Cu at (192.2, 105.0)
- added U5: ACS758xCB, solarpump:Allegro_CB_PFF, F.Cu at (138.6, 103.1)
- added U6: LM2593HV-ADJ, solarpump:TO-263-5_TabPin3, F.Cu at (25.3, 124.3)
- added U7: LM2575S-5, solarpump:TO-263-5_TabPin3, F.Cu at (97.8, 149.1)
- added U8: LM2575S-3.3, solarpump:TO-263-5_TabPin3, F.Cu at (77.7, 149.1)
- added U9: MCP23017_SO, Package_SO:SOIC-28W_7.5x17.9mm_P1.27mm, F.Cu at (85.7, 31.1)
- C10: value 220uF 6.3V -> 1uF; footprint Capacitor_THT:C_Disc_D5.0mm_W2.5mm_P5.00mm -> Capacitor_SMD:C_0805_2012Metric_Pad1.18x1.45mm_HandSolder
- C11: value 220uF 35V -> 22uF; footprint Capacitor_THT:CP_Radial_D8.0mm_P3.50mm -> Capacitor_SMD:C_0805_2012Metric_Pad1.18x1.45mm_HandSolder
- C12, C3: footprint Capacitor_THT:C_Disc_D5.0mm_W2.5mm_P5.00mm -> Capacitor_SMD:C_0805_2012Metric_Pad1.18x1.45mm_HandSolder
- C4: value 0.1uF -> 1uF; footprint Capacitor_THT:C_Disc_D5.0mm_W2.5mm_P5.00mm -> Capacitor_SMD:C_0805_2012Metric_Pad1.18x1.45mm_HandSolder
- C5: value 220uF 35V -> 0.1uF; footprint Capacitor_THT:CP_Radial_D8.0mm_P3.50mm -> Capacitor_SMD:C_0805_2012Metric_Pad1.18x1.45mm_HandSolder
- C6, C7: value 100n -> 1uF; footprint Capacitor_THT:C_Disc_D5.0mm_W2.5mm_P5.00mm -> Capacitor_SMD:C_0805_2012Metric_Pad1.18x1.45mm_HandSolder
- C8: value 100n -> 0.1uF; footprint Capacitor_THT:C_Disc_D5.0mm_W2.5mm_P5.00mm -> Capacitor_SMD:C_0805_2012Metric_Pad1.18x1.45mm_HandSolder
- C9: value 100uF -> 1uF; footprint Capacitor_THT:C_Disc_D5.0mm_W2.5mm_P5.00mm -> Capacitor_SMD:C_0805_2012Metric_Pad1.18x1.45mm_HandSolder
- D2: value DSS20-0015B -> LED; footprint Package_TO_SOT_THT:TO-220-2_Vertical -> LED_SMD:LED_0805_2012Metric_Pad1.15x1.40mm_HandSolder
- D3: value 1N4148 -> B140-E3/5AT; footprint Diode_THT:D_DO-35_SOD27_P7.62mm_Horizontal -> Diode_SMD:D_SOD-123
- D4: value 1N4934-E3 -> B140-E3/5AT; footprint Diode_THT:D_DO-41_SOD81_P7.62mm_Horizontal -> Diode_SMD:D_SOD-123
- D6: value ON_OFF -> B140-E3/5AT; footprint LED_THT:LED_D3.0mm -> Diode_SMD:D_SOD-123
- D7: value FAULT -> B140-E3/5AT; footprint LED_THT:LED_D3.0mm -> Diode_SMD:D_SOD-123
- D8: value 1N5822 -> B140-E3/5AT; footprint Diode_THT:D_DO-201AD_P15.24mm_Horizontal -> Diode_SMD:D_SOD-123
- H1, H2, H3, H4, H5: footprint MountingHole:MountingHole_3.5mm -> MountingHole:MountingHole_4.3mm_M4
- J5: value Soldered -> Conn_DISP; footprint Connector_Wire:SolderWire-0.5sqmm_1x01_D0.9mm_OD2.1mm -> Connector_PinHeader_2.00mm:PinHeader_2x06_P2.00mm_Vertical
- J6: value Soldered -> Conn_DISP; footprint Connector_Wire:SolderWire-0.5sqmm_1x01_D0.9mm_OD2.1mm -> Connector_PinHeader_2.00mm:PinHeader_2x06_P2.00mm_Vertical; moved to B.Cu
- J8: value XLR3 Male PCB -> Flow_M; footprint Connector_Audio:Jack_XLR_Neutrik_NC3FAAH-0_Horizontal -> Connector:FanPinHeader_1x03_P2.54mm_Vertical
- J9: value XLR3 Male PCB -> Fan_M; footprint Connector_Audio:Jack_XLR_Neutrik_NC3FAAH-0_Horizontal -> Connector:FanPinHeader_1x03_P2.54mm_Vertical
- JP1: value Jmp2 -> AVDD_POW1; footprint Jumper:SolderJumper-2_P1.3mm_Bridged2Bar_Pad1.0x1.5mm -> Jumper:SolderJumper-2_P1.3mm_Bridged_Pad1.0x1.5mm
- JP2: value Jmp1 -> AVDD_POW2; footprint Jumper:SolderJumper-2_P1.3mm_Bridged2Bar_Pad1.0x1.5mm -> Jumper:SolderJumper-2_P1.3mm_Bridged_Pad1.0x1.5mm
- L1: value 33uH -> 68uH; footprint Inductor_THT:L_Toroid_Vertical_L17.8mm_W8.1mm_P7.62mm_Bourns_5700 -> Inductor_THT:L_Toroid_Vertical_L35.1mm_W21.1mm_P18.50mm_Vishay_TJ6
- L2: footprint Inductor_THT:L_Axial_L5.0mm_D3.6mm_P10.00mm_Horizontal_Murata_BL01RN1A2A2 -> Inductor_SMD:L_10.4x10.4_H4.8
- MCU1: footprint RP2040_Stamp:RP2040_Stamp_SMD -> RP2040_Stamp:RP2040_Stamp_THT
- Q1: value IRLB8721PBF -> IPP019N08NF2S
- Q2, Q3: value 2N3904 -> IPP019N08NF2S; footprint Package_TO_SOT_THT:TO-92_Inline -> Package_TO_SOT_THT:TO-220-3_Vertical
- Q4, Q5: value IRLB8721PBF -> Si2306BDS; footprint Package_TO_SOT_THT:TO-220-3_Vertical -> Package_TO_SOT_SMD:SOT-23
- Q6: value 2N3904 -> Si2306BDS; footprint Package_TO_SOT_THT:TO-92_Inline -> Package_TO_SOT_SMD:SOT-23
- Q8: value 2N3904 -> IRLB8721PBF; footprint Package_TO_SOT_THT:TO-92_Inline -> Package_TO_SOT_THT:TO-220-3_Vertical
- R1: value 10K -> 4.7k; footprint Resistor_THT:R_Axial_DIN0207_L6.3mm_D2.5mm_P7.62mm_Horizontal -> Resistor_SMD:R_0805_2012Metric_Pad1.20x1.40mm_HandSolder
- R11, R26: value 10K -> 0; footprint Resistor_THT:R_Axial_DIN0207_L6.3mm_D2.5mm_P7.62mm_Horizontal -> Resistor_SMD:R_0805_2012Metric_Pad1.20x1.40mm_HandSolder
- R12, R14: value 2K2 -> 10k; footprint Resistor_THT:R_Axial_DIN0207_L6.3mm_D2.5mm_P7.62mm_Horizontal -> Resistor_SMD:R_0805_2012Metric_Pad1.20x1.40mm_HandSolder
- R13, R4, R9: value 3mOhm, 1W -> 10k; footprint solarpump:Yageo Shunt Resistor 10x5.2mm -> Resistor_SMD:R_0805_2012Metric_Pad1.20x1.40mm_HandSolder
- R15: value 2K2 -> 22k; footprint Resistor_THT:R_Axial_DIN0207_L6.3mm_D2.5mm_P7.62mm_Horizontal -> Resistor_SMD:R_0805_2012Metric_Pad1.20x1.40mm_HandSolder
- R16: value 2K2 -> 1k; footprint Resistor_THT:R_Axial_DIN0207_L6.3mm_D2.5mm_P7.62mm_Horizontal -> Resistor_SMD:R_0805_2012Metric_Pad1.20x1.40mm_HandSolder
- R17, R8: value 220 -> 10k; footprint Resistor_THT:R_Axial_DIN0207_L6.3mm_D2.5mm_P7.62mm_Horizontal -> Resistor_SMD:R_0805_2012Metric_Pad1.20x1.40mm_HandSolder
- R18: value 220 -> 4.7k; footprint Resistor_THT:R_Axial_DIN0207_L6.3mm_D2.5mm_P7.62mm_Horizontal -> Resistor_SMD:R_0805_2012Metric_Pad1.20x1.40mm_HandSolder
- R19: value 39K -> 4.7k; footprint Resistor_THT:R_Axial_DIN0207_L6.3mm_D2.5mm_P7.62mm_Horizontal -> Resistor_SMD:R_0805_2012Metric_Pad1.20x1.40mm_HandSolder
- R2: value 3mOhm, 1W -> 4.7k; footprint solarpump:Yageo Shunt Resistor 10x5.2mm -> Resistor_SMD:R_0805_2012Metric_Pad1.20x1.40mm_HandSolder
- R20: value 22K -> 10k; footprint Resistor_THT:R_Axial_DIN0207_L6.3mm_D2.5mm_P7.62mm_Horizontal -> Resistor_SMD:R_0805_2012Metric_Pad1.20x1.40mm_HandSolder
- R21, R25, R28, R29, R7: value 10K -> 10k; footprint Resistor_THT:R_Axial_DIN0207_L6.3mm_D2.5mm_P7.62mm_Horizontal -> Resistor_SMD:R_0805_2012Metric_Pad1.20x1.40mm_HandSolder
- R22, R23: value 39K -> 10k; footprint Resistor_THT:R_Axial_DIN0207_L6.3mm_D2.5mm_P7.62mm_Horizontal -> Resistor_SMD:R_0805_2012Metric_Pad1.20x1.40mm_HandSolder
- R5: value 4K7 -> 47k; footprint Resistor_THT:R_Axial_DIN0207_L6.3mm_D2.5mm_P7.62mm_Horizontal -> Resistor_SMD:R_0805_2012Metric_Pad1.20x1.40mm_HandSolder
- R6: value 4K7 -> 1k; footprint Resistor_THT:R_Axial_DIN0207_L6.3mm_D2.5mm_P7.62mm_Horizontal -> Resistor_SMD:R_0805_2012Metric_Pad1.20x1.40mm_HandSolder
- SW1: value Rotary_Encoder_Switch -> STOP_SW; footprint Rotary_Encoder:RotaryEncoder_Alps_EC11E-Switch_Vertical_H20mm -> solarpump:Schurter_SW_MTG_PUSH-12.7mm
- U1: value IR2104 -> ADS130E08; footprint Package_DIP:DIP-8_W7.62mm_LongPads -> Package_QFP:TQFP-64_10x10mm_P0.5mm
- U2: value LTC2992 -> ACS758xCB; footprint Package_SO:MSOP-16_3x4mm_P0.5mm -> solarpump:Allegro_CB_PFF
- U3: value LTC2992 -> L6398D; footprint Package_SO:MSOP-16_3x4mm_P0.5mm -> Package_SO:SOIC-8_3.9x4.9mm_P1.27mm
- U4: value LM2576HVS-5 -> TME 1212S; footprint Package_TO_SOT_SMD:TO-263-5_TabPin3 -> solarpump:TME-1212S
- moved R13 189.4 mm to (18.9, 142.2), turned to 0 degrees
- moved Q3 180.0 mm to (19.7, 138.7)
- moved SW1 172.2 mm to (62.7, 24.6), turned to 0 degrees
- moved H4 167.4 mm to (59.8, 155.3)
- moved Q6 149.2 mm to (65.8, 41.1)
- moved R28 147.2 mm to (50.2, 119.6)
- moved D6 146.1 mm to (61.0, 126.2)
- moved U4 143.9 mm to (71.3, 93.9), turned to -90 degrees
- moved R12 141.5 mm to (30.4, 136.2), turned to 0 degrees
- moved R29 140.0 mm to (45.5, 119.6)
- moved L2 139.7 mm to (74.1, 118.5), turned to 90 degrees
- moved R20 138.4 mm to (69.0, 22.6), turned to 180 degrees
- moved D8 137.9 mm to (85.8, 134.4)
- moved R21 134.6 mm to (69.6, 41.1), turned to 90 degrees
- moved R18 124.5 mm to (104.7, 27.6), turned to -90 degrees
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Connections:
- C10 pad 1: /Controller/x5V -> GND
- C10 pad 2: GND -> Net-(C10-Pad2)
- C11 pad 1: /Sol -> GND
- C11 pad 2: GND -> Net-(C11-Pad2)
- C12 pad 2: 5V -> Net-(C12-Pad2)
- C3 pad 1: /CpFET_Load -> GND
- C3 pad 2: Net-(C3-Pad2) -> /MCU/A3V3
- C4 pad 1: /CpFET_Load -> GND
- C4 pad 2: Net-(C4-Pad2) -> /MCU/A3V3
- C5 pad 1: 12V -> GND
- C5 pad 2: GND -> Net-(C5-Pad2)
- C6 pad 1: /Controller/GPIO4 -> GND
- C6 pad 2: GND -> Net-(C5-Pad2)
- C7 pad 1: /Controller/GPIO3 -> GND
- C7 pad 2: GND -> +3V3
- C8 pad 1: /Controller/GPIO2 -> GND
- C8 pad 2: GND -> +3V3
- C9 pad 2: 12V -> Net-(C9-Pad2)
- D2 pad 1: Net-(Q4-Pad2) -> /MPPT/SOLR_IN_M
- D2 pad 2: Net-(R2-Pad1) -> Net-(D2-Pad2)
- D3 pad 1: Net-(C3-Pad2) -> /MPPT/MPPT_Hvg
- D3 pad 2: 12V -> Net-(D3-Pad2)
- D4 pad 1: /PumpHi -> /MPPT/MPPT_Lvg
- D4 pad 2: /PumpLo -> Net-(D4-Pad2)
- D6 pad 2: Net-(D6-Pad2) -> GND
- D7 pad 2: Net-(D7-Pad2) -> GND
- J5 pad 1: BatTh_A -> +3V3
- J6 pad 1: BatTh_B -> /FrontPanel/FP_3V3
- J8 pad 2: /Sol -> +5V
- J8 pad 3: unconnected-(J8-Pad3) -> Net-(J8-Pad3)
- J9 pad 1: Net-(-Bat1-Pad1) -> Net-(J9-Pad1)
- J9 pad 2: /Bat -> +5V
- J9 pad 3: unconnected-(J9-Pad3) -> /MCU/Fan_Pwm
- JP1 pad 1: PuTh_A -> +3V3
- JP1 pad 2: GND -> /MCU/A3V3
- JP2 pad 1: BatTh_A -> +3V3
- JP2 pad 2: GND -> Net-(C5-Pad2)
- L1 pad 1: 12V -> MPPT_Com
- L1 pad 2: /CpFET_Load -> MPPT_OUT
- L2 pad 1: /Controller/x5V -> Net-(D6-Pad1)
- L2 pad 2: Net-(D8-Pad1) -> +12V
- MCU1 pad 1: /Controller/LTC2_G1 -> /MCU/Fan_En+
- MCU1 pad 10: PuFET -> /MCU/MPPT_PWMhi
- MCU1 pad 11: CpFET_A -> /MCU/MPPT_PWMlo
- MCU1 pad 12: CpFET_B -> Net-(MCU1-Pad12)
- MCU1 pad 13: /Controller/SPI_MISO -> Net-(MCU1-Pad13)
- MCU1 pad 14: /Controller/SPI_CS -> Net-(MCU1-Pad14)
- MCU1 pad 15: /Controller/SPI_CLK -> Net-(MCU1-Pad15)
- MCU1 pad 16: /Controller/SPI_MOSI -> Net-(MCU1-Pad16)
- MCU1 pad 17: /Controller/GPIO1 -> /MCU/BUCK_PWMlo
- MCU1 pad 18: /Controller/GPIO2 -> /MCU/BUCK_PWMhi
- MCU1 pad 19: /Controller/GPIO3 -> /MCU/I2C_INT
- MCU1 pad 2: /Controller/LTC2_G2 -> unconnected-(MCU1-Pad2)
- MCU1 pad 20: /Controller/GPIO4 -> /MCU/UART_ST
- MCU1 pad 21: unconnected-(MCU1-Pad21) -> /MCU/UART_TX
- MCU1 pad 22: unconnected-(MCU1-Pad22) -> /MCU/UART_RX
- MCU1 pad 23: /Controller/FlowPWM_3V3 -> /MCU/Enable_Aux
- MCU1 pad 24: unconnected-(MCU1-Pad24) -> /MCU/Enable_Pump
- MCU1 pad 25: Net-(D6-Pad2) -> /MCU/Fan_Pwm
- MCU1 pad 26: Net-(D7-Pad2) -> /MCU/Flow_Sig
- MCU1 pad 27: BatTh_B -> unconnected-(MCU1-Pad27)
- MCU1 pad 28: PuTh_B -> Net-(MCU1-Pad28)
- MCU1 pad 29: unconnected-(MCU1-Pad29) -> Net-(MCU1-Pad29)
- MCU1 pad 3: /Controller/LTC1_G1 -> /MCU/SPI_CLK
- MCU1 pad 30: unconnected-(MCU1-Pad30) -> Net-(MCU1-Pad30)
- MCU1 pad 32: VBAT -> unconnected-(MCU1-Pad32)
- MCU1 pad 33: 5V -> +5V
- MCU1 pad 34: /Controller/3V3 -> unconnected-(MCU1-Pad34)
- MCU1 pad 35: USB_D- -> /MCU/USB_D-
- MCU1 pad 36: USB_D+ -> /MCU/USB_D+
- MCU1 pad 4: /Controller/LTC1_G2 -> /MCU/SPI_MOSI
- MCU1 pad 40: unconnected-(MCU1-Pad40) -> /MCU/~{RESET}
- MCU1 pad 5: /Controller/SDA_0 -> /MCU/SPI_MISO
- MCU1 pad 6: /Controller/SCL_0 -> /MCU/SPI_CS
- MCU1 pad 7: unconnected-(MCU1-Pad7) -> /MCU/I2C_SDA
- MCU1 pad 8: unconnected-(MCU1-Pad8) -> /MCU/I2C_SCL
- MCU1 pad 9: BatFET -> /MCU/MPPT_BACKen
- Q1 pad 1: Net-(Q1-Pad1) -> /MPPT/BACK_gate
- Q1 pad 2: Net-(-Bat1-Pad1) -> MPPT_IN
- Q1 pad 3: GND -> /MPPT/SOLR_IN_M
- Q2 pad 1: Net-(Q1-Pad1) -> Net-(D3-Pad2)
- Q2 pad 2: BatFET -> MPPT_IN
- Q2 pad 3: Net-(Q2-Pad3) -> MPPT_Com
- Q3 pad 1: /CpFET_Drv_A -> Net-(D4-Pad2)
- Q3 pad 2: CpFET_A -> MPPT_Com
- Q3 pad 3: Net-(Q3-Pad3) -> GND
- Q4 pad 1: /CpFET_Drv_A -> /MCU/MPPT_BACKen
- Q4 pad 2: Net-(Q4-Pad2) -> GND
- Q4 pad 3: /CpFET_Load -> Net-(C19-Pad1)
- Q5 pad 1: /CpFET_Drv_B -> /MCU/Fan_En+
- Q5 pad 2: /CpFET_Load -> GND
- Q5 pad 3: GND -> Net-(J9-Pad1)
- Q6 pad 1: Net-(Q6-Pad1) -> /FrontPanel/BUZZER
- Q6 pad 2: PuFET -> /FrontPanel/FP_GND
- Q6 pad 3: Net-(Q6-Pad3) -> Net-(BZ1-Pad2)
- Q7 pad 1: Net-(Q6-Pad1) -> Net-(D9-Pad2)
- Q7 pad 2: /PumpLo -> /BATTERY/Load_P
- Q7 pad 3: GND -> /OUTPUT/OUT_Com
- Q8 pad 1: /CpFET_Drv_B -> Net-(D10-Pad2)
- Q8 pad 2: CpFET_B -> /OUTPUT/OUT_Com
- Q8 pad 3: Net-(Q8-Pad3) -> GND
- R1 pad 1: /Bat -> /MCU/A3V3
- R1 pad 2: Net-(Q2-Pad3) -> /MCU/A1V66
- R11 pad 1: /PumpHi -> Net-(D4-Pad2)
- R11 pad 2: Net-(Q6-Pad3) -> /MPPT/MPPT_Lvg
- R12 pad 1: CpFET_B -> Net-(D3-Pad2)
- R12 pad 2: GND -> MPPT_Com
- R13 pad 1: 5V -> Net-(D4-Pad2)
- R13 pad 2: Net-(R13-Pad2) -> GND
- R14 pad 1: CpFET_A -> /MCU/MPPT_BACKen
- R15 pad 1: PuFET -> MPPT_OUT
- R15 pad 2: GND -> /MCU/VLoad+
- R16 pad 1: BatFET -> /MCU/VLoad+
- R17 pad 1: Net-(D6-Pad1) -> /MCU/Fan_En+
- R18 pad 1: Net-(D7-Pad1) -> /FrontPanel/FP_3V3
- R18 pad 2: GND -> /FrontPanel/I2C_SDA
- R19 pad 1: /Controller/3V3 -> /FrontPanel/FP_3V3
- R19 pad 2: PuTh_B -> /FrontPanel/I2C_SCL
- R2 pad 1: Net-(R2-Pad1) -> /MCU/A1V66
- R2 pad 2: SolShuntB -> GNDA
- R20 pad 1: FlowPWM_5V -> Net-(R20-Pad1)
- R20 pad 2: /Controller/FlowPWM_3V3 -> /FrontPanel/FP_3V3
- R21 pad 1: GND -> /FrontPanel/BUZZER
- R21 pad 2: Net-(Q6-Pad1) -> /FrontPanel/FP_GND
- R22 pad 1: /Controller/FlowPWM_3V3 -> /FrontPanel/FP_3V3
- R22 pad 2: GND -> /FrontPanel/ROT_SW
- R23 pad 1: /Controller/3V3 -> /FrontPanel/FP_3V3
- R23 pad 2: BatTh_B -> /FrontPanel/ROT_B
- R25 pad 1: 12V -> /MCU/BUCK_PWMhi
- R25 pad 2: Net-(Q3-Pad3) -> GND
- R26 pad 1: GND -> Net-(D9-Pad2)
- R26 pad 2: /CpFET_Drv_A -> /OUTPUT/OUT_Hvg
- R28 pad 1: 12V -> Net-(D9-Pad2)
- R28 pad 2: Net-(Q8-Pad3) -> /OUTPUT/OUT_Com
- R29 pad 1: GND -> Net-(D10-Pad2)
- R29 pad 2: /CpFET_Drv_B -> GND
- R4 pad 1: 12V -> /MCU/Flow_Sig
- R4 pad 2: BatShuntB -> GND
- R5 pad 1: /Controller/3V3 -> /MPPT/SOLR_IN_M
- R5 pad 2: /Controller/SDA_0 -> /MCU/VSolr+
- R6 pad 1: /Controller/3V3 -> /MCU/VSolr+
- R6 pad 2: /Controller/SCL_0 -> GND
- R7 pad 1: GND -> /MCU/MPPT_PWMhi
- R7 pad 2: Net-(Q1-Pad1) -> GND
- R8 pad 1: 12V -> /MPPT/BACK_gate
- R8 pad 2: Net-(C4-Pad2) -> Net-(D2-Pad2)
- R9 pad 1: /PumpHi -> /MPPT/BACK_gate
- R9 pad 2: PuShuntA -> /MPPT/SOLR_IN_M
- U1 pad 1: 12V -> /MCU/A1V66
- U1 pad 2: CpFET_A -> /MCU/VCurrent_Output
- U1 pad 3: CpFET_B -> /MCU/A1V66
- U1 pad 4: GND -> /MCU/VOutput+
- U1 pad 5: /CpFET_Drv_B -> /MCU/A1V66
- U1 pad 6: /CpFET_Load -> /MCU/VCurrent_Load
- U1 pad 7: /CpFET_Drv_A -> /MCU/A1V66
- U1 pad 8: Net-(C3-Pad2) -> /MCU/VLoad+
- U2 pad 1: Net-(R13-Pad2) -> +3V3
- U2 pad 2: Net-(R13-Pad3) -> GND
- U2 pad 3: /Controller/LTC1_G1 -> /MCU/VCurrent_Solr
- U2 pad 4: unconnected-(U2-Pad4) -> /MPPT/SOLR_IN_M
- U2 pad 5: GND -> /MPPT/SOLR_IN_F
- U3 pad 1: SolShuntB -> +12V
- U3 pad 2: SolShuntA -> /MCU/MPPT_PWMhi
- U3 pad 3: /Controller/LTC2_G1 -> /MCU/MPPT_PWMlo
- U3 pad 4: unconnected-(U3-Pad4) -> GND
- U3 pad 5: GND -> /MPPT/MPPT_Lvg
- U3 pad 6: GND -> MPPT_Com
- U3 pad 7: /Controller/3V3 -> /MPPT/MPPT_Hvg
- U3 pad 8: /Controller/3V3 -> Net-(C17-Pad1)
- U4 pad 1: 12V -> Net-(C19-Pad1)
- U4 pad 2: Net-(D8-Pad1) -> +12V
- U4 pad 3: GND -> /MPPT/SOLR_IN_M
- U4 pad 4: /Controller/x5V -> /MPPT/BACK_gate
Routing:
- net +12V: track 0.00 -> 546.2 mm, vias 0 -> 6
- net +3V3: track 0.00 -> 500.6 mm, vias 0 -> 7
- net +5V: track 0.00 -> 228.4 mm, vias 0 -> 1
- net 5V: track 179.8 -> 0.00 mm, vias 1 -> 0
- net /MCU/VCurrent_Solr: track 0.00 -> 176.1 mm, vias 0 -> 3
- net /FrontPanel/FP_3V3: track 0.00 -> 171.6 mm, vias 0 -> 2
- net /MCU/MPPT_BACKen: track 0.00 -> 168.6 mm, vias 0 -> 2
- net 12V: track 161.9 -> 0.00 mm, vias 2 -> 0
- net /BATTERY/Load_P: track 0.00 -> 158.0 mm, vias 0 -> 2
- net /MPPT/SOLR_IN_M: track 0.00 -> 137.3 mm, vias 0 -> 2
- net /MCU/MPPT_PWMhi: track 0.00 -> 135.2 mm, vias 0 -> 2
- net /FrontPanel/ROT_SW: track 0.00 -> 131.0 mm, vias 0 -> 1
- net /MCU/MPPT_PWMlo: track 0.00 -> 119.5 mm, vias 0 -> 2
- net /MCU/Enable_Pump: track 0.00 -> 113.5 mm, vias 0 -> 4
- net /OUTPUT/OUT_Com: track 0.00 -> 112.4 mm, vias 0 -> 4
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- added copper zone on B.Cu, net /FrontPanel/FP_GND
- added copper zone on F.Cu, net /FrontPanel/FP_GND
- added copper zone on F.Cu, net GND
- added copper zone on F.Cu, net GNDA
Other:
- board size 116.5 x 66 mm -> 175.1 x 146.4 mm
- board text added: "0.2500 mm / 0.0000 mm"
- board text added: "0.3000 mm"
- board text added: "1.6000 mm"
- board text added: "12V 5V 3V3 GND"
- board text added: "175.2660 mm x 146.6178 mm"
- board text added: "2"
- board text added: "3V3 MOSI CS CLK MISO GND SCL SDA INT RST 3V3 GND"
- board text added: "BOARD CHARACTERISTICS"
- board text added: "Board Thickness:"
- board text added: "Board overall dimensions:"
- board text added: "Castellated pads:"
- board text added: "Copper Finish:"
- board text added: "Copper Layer Count:"
- board text added: "Edge card connectors:"
- board text added: "Fan"
- board text added: "Flow"
- board text added: "Front Panel"
- board text added: "GND 5V PWM"
- board text added: "GND 5V SIG"
- board text added: "Impedance Control:"
- board text added: "JLCJLCJLCJLC"
- board text added: "Min hole diameter:"
- board text added: "Min track/spacing:"
- board text added: "No"
- board text added: "None"
- board text added: "Plated Board Edge:"
- board text added: "ST TX RX"
- board text added: "SolarPump V3 Ruth Ivimey-Cook 2021 Board: D 1.0"
- board text added: "SolarPump V3 Ruth Ivimey-Cook 2021 Board: P 1.0"
- board text added: "SolrIn OutPmp OutAux Battery + - + - + - + -"
- board text added: "Thanks: ASCAS/TechBuilder 1KW WiFi MPPT Solar Charger"
- board text added: "USB Host"
- board text removed: "12V AGM"
- board text removed: "3V3 LiPo"
- board text removed: "5V USB"
- board text removed: "Batt SW"
- board text removed: "EXT Charger"
- board text removed: "ExtChg SW"
- board text removed: "PUMP & SENSORS"
- board text removed: "Pump SW"
- board text removed: "SPI LCD"
- board text removed: "Solar Power"
- board text removed: "Solar SW"
- board text removed: "SolarPump rev 1 (c) IvimeyCom 2021"
- board text removed: "TCH I/F"
- board text removed: "To MPPT PU1012EU"
