File: solarpump.kicad_pcb (KiCad board)
At the start: 2 copper layers, 174.6 x 156.5 mm, 247 parts, among them J1 8-way_Screw, J11 OLED_SOG320132A_M383, J12 Stemma-QT_QWIIC, J13 JST SM03B-SRSS-TB, J14 Gnd, J15 3v3, J16 AT85_PROG, J17 USB_B_Micro, J2 UART_IO, J3 AUX_POWER, J4 USB_A, J5 Conn_DISP, J6 Conn_DISP, J8 Flow_M, J9 Fan_M, M3 Pico_Display_Pack, Q1 IPP019N08NF2S, Q10 Si2306BDS, Q11 IRLB8721PBF, Q12 IRLB8721PBF, Q2 IPP019N08NF2S, Q3 IPP019N08NF2S, Q4 Si2306BDS, Q5 Si2306BDS, Q6 Si2306BDS, Q7 IRLB8721PBF, Q8 IRLB8721PBF, Q9 Si2306BDS, SW1 STOP_SW, SW2 Rotary Enc EC11E, SW3 SW_A, SW4 SW_B, SW5 SW_X, SW6 SW_Y, SW7 ~{BOOTSEL}, U1 AT24C040, U10 MCP23017_SO, U11 L6398D, U12 ACS758xCB, U13 ACS758xCB, U14 DS3231, U15 ATtiny85-20S, U2 ADS130E08, U3 ACS758xCB, U4 L6398D, U5 TME 1212S, U6 ACS758xCB, U7 LM2593HVS-ADJ, U8 LM2575S-5, U9 LM2575S-3.3

Commit message: Further works...
Parts:
- removed BZ1: Buzzer, solarpump:Buzzer_3V
- removed C57: 0.1uF, Capacitor_SMD:C_0805_2012Metric_Pad1.18x1.45mm_HandSolder
- removed the D17 at (170.9, 43.7)
- removed the G*** at (57.0, 128.1)
- removed HS5, HS6, HS7: HSink, MountingHole:MountingHole_2.7mm_M2.5_Pad_Via
- removed the J9 at (88.0, 158.9)
- removed M3: Pico_Display_Pack, solarpump:DIP-40_W17.78mm_Socket
- removed MCU1: RP2040_Stamp_W, IvimeyCom:RP2040_Stamp_THT
- removed NT1: NetTie_2, NetTie:NetTie-2_SMD_Pad2.0mm
- removed the Q9 at (98.2, 82.0)
- removed the R61 at (53.1, 158.6)
- removed the R63 at (115.4, 131.6)
- removed RN1: RNet03_10K, Resistor_THT:R_Array_SIP4
- removed the TP1 at (105.9, 154.9)
- removed TP10: GPIO3, TestPoint:TestPoint_Pad_1.0x1.0mm
- removed TP2: VTEST-, TestPoint:TestPoint_Pad_1.0x1.0mm
- removed TP3: GBP1_TP, TestPoint:TestPoint_Pad_1.0x1.0mm
- removed TP4: GBP2_TP, TestPoint:TestPoint_Pad_1.0x1.0mm
- removed TP6: AT85_INT, TestPoint:TestPoint_Pad_1.0x1.0mm
- removed TP7: GPIO1, TestPoint:TestPoint_Pad_1.0x1.0mm
- removed TP8: GPIO2, TestPoint:TestPoint_Pad_1.0x1.0mm
- removed TP9: GPIO4, TestPoint:TestPoint_Pad_1.0x1.0mm
- added BT1: Li-Ion 3V7, Connector_JST:JST_PH_B2B-PH-K_1x02_P2.00mm_Vertical, F.Cu at (189.9, 87.6)
- added C100: 1uF, Capacitor_SMD:C_0603_1608Metric, F.Cu at (415.1, 150.8)
- added C101: 0.1uF, Capacitor_SMD:C_0402_1005Metric, F.Cu at (398.6, 147.3)
- added C102: 0.1uF, Capacitor_SMD:C_0402_1005Metric, F.Cu at (413.0, 153.2)
- added C103: 1uF, Capacitor_SMD:C_0603_1608Metric, F.Cu at (411.8, 153.7)
- added C104: 12pF, Capacitor_SMD:C_0402_1005Metric, F.Cu at (404.1, 145.3)
- added C105: 12pF, Capacitor_SMD:C_0402_1005Metric, F.Cu at (399.7, 145.3)
- added C106: 0.1uF, Capacitor_SMD:C_0402_1005Metric, F.Cu at (232.1, 129.6)
- added C107: 0.1uF, Capacitor_SMD:C_0402_1005Metric, F.Cu at (230.2, 129.6)
- added C108: 0.1uF, Capacitor_SMD:C_0402_1005Metric, F.Cu at (231.9, 122.7)
- added C109: 0.1uF,100V, Capacitor_SMD:C_0805_2012Metric_Pad1.18x1.45mm_HandSolder, F.Cu at (221.5, 127.7)
- added C110: 0.1uF,100V, Capacitor_SMD:C_0805_2012Metric_Pad1.18x1.45mm_HandSolder, F.Cu at (217.3, 119.0)
- added C111: 0.1uF,100V Tant, Capacitor_SMD:C_0805_2012Metric_Pad1.18x1.45mm_HandSolder, F.Cu at (192.0, 187.5)
- added C112: 0.1uF,100V Tant, Capacitor_SMD:C_0805_2012Metric_Pad1.18x1.45mm_HandSolder, F.Cu at (191.7, 166.3)
- added C113: 0.1uF,100V Tant, Capacitor_SMD:C_0805_2012Metric_Pad1.18x1.45mm_HandSolder, F.Cu at (192.0, 158.2)
- added C114: 0.1uF,100V Tant, Capacitor_SMD:C_0805_2012Metric_Pad1.18x1.45mm_HandSolder, F.Cu at (191.7, 136.7)
- added C115: 0.1uF,100V Tant, Capacitor_SMD:C_0805_2012Metric_Pad1.18x1.45mm_HandSolder, F.Cu at (192.0, 129.0)
- added C116: 0.1uF,100V Tant, Capacitor_SMD:C_0805_2012Metric_Pad1.18x1.45mm_HandSolder, F.Cu at (191.7, 107.6)
- added C117: 10uF, Capacitor_SMD:C_0603_1608Metric, F.Cu at (188.9, 23.9)
- added C118: 0.1uF, Capacitor_SMD:C_0603_1608Metric, F.Cu at (188.4, 30.4)
- added C119: 100uF, Capacitor_SMD:C_0603_1608Metric, F.Cu at (180.6, 20.2)
- added C120: 10uF, Capacitor_SMD:C_0603_1608Metric, F.Cu at (185.5, 23.9)
- added C24: 0.1uF, Capacitor_SMD:C_0603_1608Metric, F.Cu at (70.5, 227.4)
- added C35: 0.1uF, Capacitor_SMD:C_0402_1005Metric, F.Cu at (92.7, 228.8)
- added C50: 0.1uF, Capacitor_SMD:C_0603_1608Metric, F.Cu at (205.0, 95.2)
- added C53: 4.7uF,25V, Capacitor_SMD:C_0805_2012Metric_Pad1.18x1.45mm_HandSolder, F.Cu at (213.5, 77.7)
- added C60: 4.7uF, Capacitor_SMD:C_0603_1608Metric, F.Cu at (194.3, 91.8)
- added C61: 10uF, Capacitor_SMD:C_0603_1608Metric, F.Cu at (189.4, 34.4)
- added C63: 4.7uF,10V, Capacitor_SMD:C_0805_2012Metric_Pad1.18x1.45mm_HandSolder, F.Cu at (182.8, 83.3)
- added C66: 1uF, Capacitor_SMD:C_0603_1608Metric, F.Cu at (219.5, 17.9)
- added C67: 0.1uF, Capacitor_SMD:C_0603_1608Metric, F.Cu at (267.0, 54.6)
- added C68: 0.1uF, Capacitor_SMD:C_0603_1608Metric, F.Cu at (266.9, 51.9)
- added C70: 0.1uF, Capacitor_SMD:C_0603_1608Metric, F.Cu at (266.9, 49.0)
- added C72: 0.1uF, Capacitor_SMD:C_0603_1608Metric, F.Cu at (266.9, 46.2)
- added C75: 0.1uF, Capacitor_SMD:C_0603_1608Metric, F.Cu at (295.3, 40.2)
- added C76: 0.1uF, Capacitor_SMD:C_0603_1608Metric, F.Cu at (296.9, 37.2)
- added C77: 0.1uF, Capacitor_SMD:C_0603_1608Metric, F.Cu at (323.6, 38.5)
- added C79: 0.1uF, Capacitor_SMD:C_0603_1608Metric, F.Cu at (375.1, 137.8)
- added C80: 0.1uF, Capacitor_SMD:C_0603_1608Metric, F.Cu at (364.2, 152.7)
- added C81: 0.1uF, Capacitor_SMD:C_0603_1608Metric, F.Cu at (362.2, 152.7)
- added C82: 0.1uF, Capacitor_SMD:C_0603_1608Metric, F.Cu at (344.4, 156.7)
- added C83: 2nF, 50V, Low ESR, Capacitor_SMD:C_0805_2012Metric_Pad1.18x1.45mm_HandSolder, F.Cu at (342.0, 120.9)
- added C84: 22uF,>35V, Capacitor_Tantalum_SMD:CP_EIA-7360-38_Kemet-E, F.Cu at (355.0, 78.8)
- added C85: 22uF,>35V, Capacitor_Tantalum_SMD:CP_EIA-7360-38_Kemet-E, F.Cu at (347.9, 78.8)
- added C86: 22uF,>35V, Capacitor_Tantalum_SMD:CP_EIA-7360-38_Kemet-E, F.Cu at (362.0, 78.8)
- added C87: 0.1uF, Capacitor_SMD:C_0603_1608Metric, F.Cu at (349.4, 156.7)
- added C88: 0.1uF, Capacitor_SMD:C_0603_1608Metric, F.Cu at (347.2, 156.7)
- added C89: 0.1uF, Capacitor_SMD:C_0603_1608Metric, F.Cu at (357.2, 93.2)
- added C90: 0.1uF, Capacitor_SMD:C_0402_1005Metric, F.Cu at (345.9, 152.0)
- added C91: 0.1uF, Capacitor_SMD:C_0402_1005Metric, F.Cu at (415.6, 137.3)
- added C92: 0.1uF, Capacitor_SMD:C_0402_1005Metric, F.Cu at (356.7, 94.4)
- added C93: 0.1uF, Capacitor_SMD:C_0402_1005Metric, F.Cu at (416.7, 149.6)
- added C94: 0.1uF, Capacitor_SMD:C_0402_1005Metric, F.Cu at (340.2, 151.3)
- added C95: 0.1uF, Capacitor_SMD:C_0402_1005Metric, F.Cu at (409.1, 141.5)
- added C96: 0.1uF, Capacitor_SMD:C_0402_1005Metric, F.Cu at (399.7, 147.3)
- added C97: 0.1uF, Capacitor_SMD:C_0402_1005Metric, F.Cu at (412.0, 151.7)
- added C98: 0.1uF, Capacitor_SMD:C_0402_1005Metric, F.Cu at (408.8, 152.4)
- added C99: 0.1uF, Capacitor_SMD:C_0402_1005Metric, F.Cu at (413.9, 142.0)
- added D14: Orange,160mcd, LED_SMD:LED_1206_3216Metric_Pad1.42x1.75mm_HandSolder, F.Cu at (192.4, 77.2)
- added D22: SMAJ54CA, Diode_SMD:D_SMA, F.Cu at (375.8, 96.9)
- added D23: SMAJ54CA, Diode_SMD:D_SMA, F.Cu at (375.8, 112.3)
- added D24: Red,150mcd, LED_SMD:LED_1206_3216Metric_Pad1.42x1.75mm_HandSolder, F.Cu at (309.5, 144.1)
- added D25: Red,150mcd, LED_SMD:LED_1206_3216Metric_Pad1.42x1.75mm_HandSolder, F.Cu at (357.9, 143.8)
- added D26: B150-E3,50V, Diode_SMD:D_SMA, F.Cu at (231.8, 118.6)
- added D27: B150-E3,50V, Diode_SMD:D_SMA, F.Cu at (218.7, 126.1)
- added D28: SMAJ54CA, Diode_SMD:D_SMA, F.Cu at (231.8, 111.1)
- added D29: Red,150mcd, LED_SMD:LED_1206_3216Metric_Pad1.42x1.75mm_HandSolder, F.Cu at (188.6, 186.0)
- added D30: Red,150mcd, LED_SMD:LED_1206_3216Metric_Pad1.42x1.75mm_HandSolder, F.Cu at (188.6, 165.9)
- added D31: Red,150mcd, LED_SMD:LED_1206_3216Metric_Pad1.42x1.75mm_HandSolder, F.Cu at (188.6, 156.7)
- added D32: Red,150mcd, LED_SMD:LED_1206_3216Metric_Pad1.42x1.75mm_HandSolder, F.Cu at (188.6, 136.8)
- added D33: Red,150mcd, LED_SMD:LED_1206_3216Metric_Pad1.42x1.75mm_HandSolder, F.Cu at (188.6, 127.5)
- added D34: Red,150mcd, LED_SMD:LED_1206_3216Metric_Pad1.42x1.75mm_HandSolder, F.Cu at (188.8, 107.8)
- added DZ1: BZV90-C30, Package_TO_SOT_SMD:SOT-223-3_TabPin2, F.Cu at (80.2, 163.5)
- added F3: Fuse 25A, Fuse:Fuse_Schurter_UMZ250, F.Cu at (365.3, 97.8)
- added F4: Fuse 25A, Fuse:Fuse_Schurter_UMZ250, F.Cu at (365.4, 121.7)
- added F5: Fuse 25A, Fuse:Fuse_Schurter_UMZ250, F.Cu at (235.5, 136.5)
- added H11: Mount, MountingHole:MountingHole_4.3mm_M4, F.Cu at (26.6, 162.6)
- added H12: Mount, MountingHole:MountingHole_4.3mm_M4, F.Cu at (26.7, 228.5)
- added H5: Mount, MountingHole:MountingHole_4.3mm_M4, F.Cu at (247.7, 78.8)
- added H6: Mount, MountingHole:MountingHole_4.3mm_M4, F.Cu at (247.7, 228.0)
- added J10: SAMTEC_ET60_24S_2Pr_Socket, solarpump:SAMTEC_ET60S-000-3-08-D02-L-R1-S, F.Cu at (304.1, 110.9)
- added J12: Gnd, TestPoint:TestPoint_Plated_Hole_D2.0mm, F.Cu at (183.6, 228.1)
- added J18: Wire_Solr_N, Connector_Wire:SolderWire-2sqmm_1x01_D2mm_OD3.9mm, F.Cu at (41.0, 229.5)
- added J19: Wire_Solr_P, Connector_Wire:SolderWire-2sqmm_1x01_D2mm_OD3.9mm, F.Cu at (41.0, 222.5)
- added J20: JST SM03B-SRSS-TB, Connector_JST:JST_SH_SM03B-SRSS-TB_1x03-1MP_P1.00mm_Horizontal, F.Cu at (116.8, 230.0)
- added J21: JST SM03B-SRSS-TB, Connector_JST:JST_SH_SM03B-SRSS-TB_1x03-1MP_P1.00mm_Horizontal, F.Cu at (109.7, 230.0)
- added J22: USB_B_Micro, Connector_USB:USB_Micro-B_Amphenol_10104110_Horizontal, F.Cu at (56.2, 228.8)
- added J23: OLED_SOG320132A_M383, solarpump:OLED_SOG320132A_M383, F.Cu at (235.9, 34.3)
- added J24: uHAT, Module:Raspberry_Pi_Zero_Socketed_THT_FaceDown_MountingHoles, B.Cu at (248.5, 48.8)
- added J26: JST SM03B-SRSS-TB, Connector_JST:JST_SH_SM03B-SRSS-TB_1x03-1MP_P1.00mm_Horizontal, F.Cu at (363.1, 145.5)
- added J27: JST SM03B-SRSS-TB, Connector_JST:JST_SH_SM03B-SRSS-TB_1x03-1MP_P1.00mm_Horizontal, F.Cu at (302.3, 145.4)
- added J28: USB_B_Micro, Connector_USB:USB_Micro-B_Amphenol_10104110_Horizontal, F.Cu at (327.9, 145.2)
- added J29: OP_Wire_Aux_P, Connector_Wire:SolderWire-2sqmm_1x01_D2mm_OD3.9mm, F.Cu at (375.0, 123.1)
- added J30: OP_Wire_Aux_N, Connector_Wire:SolderWire-2sqmm_1x01_D2mm_OD3.9mm, F.Cu at (375.0, 117.2)
- added J31: OP_Wire_Pump_P, Connector_Wire:SolderWire-2sqmm_1x01_D2mm_OD3.9mm, F.Cu at (375.0, 107.3)
- added J32: OP_Wire_Pump_N, Connector_Wire:SolderWire-2sqmm_1x01_D2mm_OD3.9mm, F.Cu at (375.0, 101.3)
- added J33: Amass_XT30PW, solarpump:Amass_XT30PW, F.Cu at (387.6, 104.2)
- added J34: Amass_XT30PW, solarpump:Amass_XT30PW, F.Cu at (387.6, 120.0)
- added J35: Screw_Terminal_01x02, Connector_Phoenix_MC_HighVoltage:PhoenixContact_MCV_1,5_2-GF-5.08_1x02_P5.08mm_Vertical_ThreadedFlange_MountHole, F.Cu at (247.3, 149.9)
- added J37: Flow_M, Connector:FanPinHeader_1x03_P2.54mm_Vertical, F.Cu at (354.0, 19.2)
- added J38: Speaker, Connector_JST:JST_PH_S2B-PH-K_1x02_P2.00mm_Horizontal, B.Cu at (184.2, 19.1)
- added J39: Buzzer, Connector_JST:JST_PH_S2B-PH-K_1x02_P2.00mm_Horizontal, F.Cu at (168.0, 50.3)
- added J41: Conn_DISP, Connector_PinHeader_2.00mm:PinHeader_2x05_P2.00mm_Vertical, F.Cu at (337.8, 15.3)
- added J42: ~, Connector_PinHeader_2.00mm:PinHeader_2x05_P2.00mm_Vertical, F.Cu at (201.5, 227.1)
- added J6: Conn_DISP, Connector_PinHeader_2.00mm:PinHeader_2x08_P2.00mm_Vertical, F.Cu at (231.7, 214.3)
- added J7: SAMTEC_ET60_24S_2Pr_Pins, solarpump:SAMTEC_ET60T-000-3-08-D02-X-R1-S, F.Cu at (247.3, 111.2)
- added M1: SPI_CAN_MOD, IvimeyCom:MCP2515 CAN module_SMD, B.Cu at (285.6, 42.6)
- added OC1: HCPL-314Js, Package_SO:SOIC-16W-12_7.5x10.3mm_P1.27mm, F.Cu at (188.1, 198.0)
- added OC2: HCPL-314Js, Package_SO:SOIC-16W-12_7.5x10.3mm_P1.27mm, F.Cu at (199.9, 198.0)
- added Q13: IRLB8721PBF, Package_TO_SOT_THT:TO-220-3_Vertical, F.Cu at (327.9, 112.0)
- added Q14: IRLB8721PBF, Package_TO_SOT_THT:TO-220-3_Vertical, F.Cu at (368.6, 86.5)
- added Q15: IRLB8721PBF, Package_TO_SOT_THT:TO-220-3_Vertical, F.Cu at (368.3, 129.1)
- added Q16: SQM120P10, Package_TO_SOT_SMD:TO-263-2, F.Cu at (224.2, 110.7)
- added Q17: BC817, Package_TO_SOT_SMD:SOT-23, F.Cu at (197.6, 175.8)
- added Q18: SQM120P10, Package_TO_SOT_SMD:TO-263-2, F.Cu at (205.8, 183.2)
- added Q19: SQM120P10, Package_TO_SOT_SMD:TO-263-2, F.Cu at (205.8, 168.4)
- added Q21: BC817, Package_TO_SOT_SMD:SOT-23, F.Cu at (197.6, 146.3)
- added Q22: SQM120P10, Package_TO_SOT_SMD:TO-263-2, F.Cu at (205.8, 153.7)
- added Q23: SQM120P10, Package_TO_SOT_SMD:TO-263-2, F.Cu at (205.8, 139.0)
- added Q24: BC817, Package_TO_SOT_SMD:SOT-23, F.Cu at (197.5, 116.9)
- added Q25: SQM120P10, Package_TO_SOT_SMD:TO-263-2, F.Cu at (205.8, 124.2)
- added Q26: SQM120P10, Package_TO_SOT_SMD:TO-263-2, F.Cu at (205.8, 109.5)
- added Q27: Si2306BDS, Package_TO_SOT_SMD:SOT-23, F.Cu at (184.7, 209.3)
- added Q6: IPP019N08NF2S, Package_TO_SOT_THT:TO-220-3_Vertical, F.Cu at (74.9, 197.6)
- added R100: 10k, Resistor_SMD:R_0603_1608Metric, F.Cu at (201.6, 175.1)
- added R101: 10k, Resistor_SMD:R_0603_1608Metric, F.Cu at (188.6, 191.2)
- added R102: 470k, Resistor_SMD:R_0603_1608Metric, F.Cu at (197.0, 183.0)
- added R103: 33k, Resistor_SMD:R_0603_1608Metric, F.Cu at (181.5, 166.0)
- added R104: 270R, Resistor_SMD:R_0603_1608Metric, F.Cu at (188.7, 37.4)
- added R105: 6.8k, Resistor_SMD:R_0603_1608Metric, F.Cu at (343.8, 18.4)
- added R106: 10k, Resistor_SMD:R_0603_1608Metric, F.Cu at (343.6, 24.1)
- added R107: 42K, Resistor_SMD:R_0603_1608Metric, F.Cu at (181.5, 156.8)
- added R108: 10k, Resistor_SMD:R_0603_1608Metric, F.Cu at (201.7, 145.9)
- added R109: 10k, Resistor_SMD:R_0603_1608Metric, F.Cu at (197.6, 191.2)
- added R110: 470k, Resistor_SMD:R_0603_1608Metric, F.Cu at (197.1, 153.5)
- added R111: 33k, Resistor_SMD:R_0603_1608Metric, F.Cu at (181.5, 136.8)
- added R112: 42K, Resistor_SMD:R_0603_1608Metric, F.Cu at (181.5, 127.6)
- added R113: 10k, Resistor_SMD:R_0603_1608Metric, F.Cu at (201.7, 116.3)
- added R114: 10k, Resistor_SMD:R_0603_1608Metric, F.Cu at (184.0, 191.2)
- added R115: 470k, Resistor_SMD:R_0603_1608Metric, F.Cu at (197.2, 124.0)
- added R116: 33k, Resistor_SMD:R_0603_1608Metric, F.Cu at (181.5, 108.0)
- added R117: 10k, Resistor_SMD:R_0603_1608Metric, F.Cu at (184.7, 213.1)
- added R118: 3K3, Resistor_SMD:R_0603_1608Metric, F.Cu at (343.8, 21.3)
- added R119: 10K, Resistor_SMD:R_0603_1608Metric, F.Cu at (187.2, 23.9)
- added R120: 10R, Resistor_SMD:R_0603_1608Metric, F.Cu at (188.4, 27.2)
- added R23: 10k, Resistor_SMD:R_0603_1608Metric, F.Cu at (69.5, 223.8)
- added R24: 4.7k,0.5%, Resistor_SMD:R_0603_1608Metric, F.Cu at (76.8, 214.6)
- added R25: 4.7k,0.5%, Resistor_SMD:R_0603_1608Metric, F.Cu at (76.8, 217.7)
- added R26: 10k, Resistor_SMD:R_0603_1608Metric, F.Cu at (66.1, 209.8)
- added R47: 10K,0.5%, Resistor_SMD:R_0603_1608Metric, F.Cu at (185.5, 74.4)
- added R48: 2K, Resistor_SMD:R_0603_1608Metric, F.Cu at (191.3, 91.8)
- added R49: 25K, Resistor_SMD:R_0603_1608Metric, F.Cu at (188.3, 91.8)
- added R51: 680R, Resistor_SMD:R_0603_1608Metric, F.Cu at (179.3, 97.9)
- added R66: 10k, Resistor_SMD:R_0603_1608Metric, F.Cu at (295.3, 37.2)
- added R67: 10k, Resistor_SMD:R_0603_1608Metric, F.Cu at (296.9, 34.0)
- added R68: 10k, Resistor_SMD:R_0603_1608Metric, F.Cu at (323.6, 35.2)
- added R71: 150R, Resistor_SMD:R_0603_1608Metric, F.Cu at (188.7, 39.2)
- added R73: 33K,1%, Resistor_SMD:R_0603_1608Metric, F.Cu at (367.4, 152.7)
- added R74: 1K,1%, Resistor_SMD:R_0603_1608Metric, F.Cu at (365.8, 152.7)
- added R75: 10k, Resistor_SMD:R_0603_1608Metric, F.Cu at (340.7, 133.0)
- added R76: 0R, Resistor_SMD:R_0603_1608Metric, F.Cu at (339.3, 122.6)
- added R77: 0R, Resistor_SMD:R_0603_1608Metric, F.Cu at (422.6, 151.4)
- added R78: 10k, Resistor_SMD:R_0603_1608Metric, F.Cu at (342.5, 122.7)
- added R79: 10k, Resistor_SMD:R_0603_1608Metric, F.Cu at (420.2, 151.4)
- added R80: 4.7k,0.5%, Resistor_SMD:R_0603_1608Metric, F.Cu at (368.8, 137.8)
- added R81: 4.7k,0.5%, Resistor_SMD:R_0603_1608Metric, F.Cu at (371.9, 137.8)
- added R82: 33K,1%, Resistor_SMD:R_0603_1608Metric, F.Cu at (361.1, 126.4)
- added R83: 1K,1%, Resistor_SMD:R_0603_1608Metric, F.Cu at (341.2, 154.4)
- added R84: 10K, Resistor_SMD:R_0603_1608Metric, F.Cu at (420.3, 142.6)
- added R85: 100R, Resistor_SMD:R_0603_1608Metric, F.Cu at (364.8, 95.2)
- added R86: 100R, Resistor_SMD:R_0603_1608Metric, F.Cu at (365.1, 128.3)
- added R87: 10k, Resistor_SMD:R_0603_1608Metric, F.Cu at (365.6, 91.6)
- added R88: 10k, Resistor_SMD:R_0603_1608Metric, F.Cu at (365.1, 131.6)
- added R89: 10K, Resistor_SMD:R_0603_1608Metric, F.Cu at (398.4, 143.1)
- added R90: 27R, Resistor_SMD:R_0603_1608Metric, F.Cu at (332.1, 142.2)
- added R91: 27R, Resistor_SMD:R_0603_1608Metric, F.Cu at (328.7, 141.8)
- added R92: 100R, Resistor_SMD:R_0603_1608Metric, F.Cu at (361.0, 141.0)
- added R93: 100R, Resistor_SMD:R_0603_1608Metric, F.Cu at (364.3, 141.0)
- added R94: 72R, Resistor_SMD:R_0603_1608Metric, F.Cu at (308.4, 142.0)
- added R95: 72R, Resistor_SMD:R_0603_1608Metric, F.Cu at (357.5, 147.2)
- added R96: 22k, Resistor_SMD:R_0603_1608Metric, F.Cu at (227.1, 130.0)
- added R97: 1k, Resistor_SMD:R_0603_1608Metric, F.Cu at (230.1, 131.0)
- added R98: 10k, Resistor_SMD:R_0603_1608Metric, F.Cu at (218.4, 121.8)
- added R99: 42K, Resistor_SMD:R_0603_1608Metric, F.Cu at (181.5, 186.2)
- added RV1: 10K, Potentiometer_SMD:Potentiometer_Bourns_TC33X_Vertical, F.Cu at (181.8, 33.8)
- added RV2: 10K, Potentiometer_SMD:Potentiometer_Bourns_TC33X_Vertical, F.Cu at (182.0, 23.9)
- added SW1: SW_RESET, Button_Switch_SMD:SW_SPST_B3U-1000P, F.Cu at (222.6, 204.1)
- added SW10: SW_SPST, PCM_4ms_Switch:Switch_Toggle_SPST_SubMini, F.Cu at (239.3, 146.0)
- added SW9: SW_RESET, Button_Switch_SMD:SW_SPST_B3U-1000P, F.Cu at (408.8, 157.3)
- added TVS1: TVS, Package_TO_SOT_SMD:SOT-23, F.Cu at (105.8, 195.3)
- added TVS10: TVS, Package_TO_SOT_SMD:SOT-23, F.Cu at (316.7, 138.0)
- added TVS11: TVS, Package_TO_SOT_SMD:SOT-23, F.Cu at (312.9, 133.7)
- added TVS2: TVS, Package_TO_SOT_SMD:SOT-23, F.Cu at (105.9, 200.0)
- added TVS3: TVS, Package_TO_SOT_SMD:SOT-23, F.Cu at (104.4, 229.0)
- added TVS4: TVS, Package_TO_SOT_SMD:SOT-23, F.Cu at (105.9, 204.7)
- added TVS5: TVS, Package_TO_SOT_SMD:SOT-23, F.Cu at (285.4, 16.5)
- added TVS6: TVS, Package_TO_SOT_SMD:SOT-23, F.Cu at (232.2, 29.5)
- added TVS7: TVS, Package_TO_SOT_SMD:SOT-23, F.Cu at (227.8, 29.5)
- added TVS8: TVS, Package_TO_SOT_SMD:SOT-23, F.Cu at (307.9, 138.5)
- added TVS9: TVS, Package_TO_SOT_SMD:SOT-23, F.Cu at (311.8, 138.5)
- added U14: RP2040, Package_DFN_QFN:QFN-56-1EP_7x7mm_P0.4mm_EP3.2x3.2mm_ThermalVias, F.Cu at (91.5, 223.1)
- added U16: LM2593HVS-ADJ, Package_TO_SOT_SMD:TO-263-7_TabPin4, F.Cu at (217.5, 93.8)
- added U17: LV2862XDDC, Package_TO_SOT_SMD:SOT-23-6, F.Cu at (185.7, 79.3)
- added U18: MCP73871-2CC, Package_DFN_QFN:QFN-20-1EP_4x4mm_P0.5mm_EP2.5x2.5mm, F.Cu at (183.9, 88.5)
- added U19: AP7361C-33ER-13, Package_TO_SOT_SMD:SOT-223-3_TabPin2, F.Cu at (190.3, 96.6)
- added U20: LM809-M3X 3.08, Package_TO_SOT_SMD:SOT-23, F.Cu at (186.7, 83.3)
- added U22: ACS71240LLCBTR-025B3, Package_SO:SOIC-8_3.9x4.9mm_P1.27mm, F.Cu at (315.7, 81.2)
- added U23: L6398D, Package_SO:SOIC-8_3.9x4.9mm_P1.27mm, F.Cu at (340.5, 127.3)
- added U24: ADS1115IDGS, Package_SO:TSSOP-10_3x3mm_P0.5mm, F.Cu at (355.9, 128.2)
- added U25: ADS131M04-PW, Package_SO:TSSOP-20_4.4x6.5mm_P0.65mm, F.Cu at (355.9, 128.2)
- added U26: ACS71240LLCBTR-025B3, Package_SO:SOIC-8_3.9x4.9mm_P1.27mm, F.Cu at (359.5, 89.5)
- added U27: SN65HVD234, Package_SO:SOIC-8_3.9x4.9mm_P1.27mm, F.Cu at (302.2, 138.9)
- added U28: W25Q32JV, Package_SON:WSON-8-1EP_6x5mm_P1.27mm_EP3.4x4mm, F.Cu at (419.0, 146.2)
- added U29: 2EDN752x, Package_SO:Infineon_PG-DSO-8-43, F.Cu at (363.8, 110.9)
- added U30: RP2040, Package_DFN_QFN:QFN-56-1EP_7x7mm_P0.4mm_EP3.2x3.2mm_ThermalVias, F.Cu at (410.1, 146.7)
- added U31: ACS71240LLCBTR-025B3, Package_SO:SOIC-8_3.9x4.9mm_P1.27mm, F.Cu at (229.0, 126.2)
- added U32: BCR430UW6, Package_TO_SOT_SMD:SC-74-6_1.55x2.9mm_P0.95mm, F.Cu at (184.8, 186.0)
- added U33: BCR430UW6, Package_TO_SOT_SMD:SC-74-6_1.55x2.9mm_P0.95mm, F.Cu at (184.8, 165.9)
- added U34: BCR430UW6, Package_TO_SOT_SMD:SC-74-6_1.55x2.9mm_P0.95mm, F.Cu at (184.8, 156.7)
- added U35: BCR430UW6, Package_TO_SOT_SMD:SC-74-6_1.55x2.9mm_P0.95mm, F.Cu at (184.8, 136.6)
- added U36: BCR430UW6, Package_TO_SOT_SMD:SC-74-6_1.55x2.9mm_P0.95mm, F.Cu at (184.8, 127.5)
- added U37: BCR430UW6, Package_TO_SOT_SMD:SC-74-6_1.55x2.9mm_P0.95mm, F.Cu at (185.0, 107.8)
- added U38: 74LVC1G125, Package_TO_SOT_SMD:SOT-23-5, F.Cu at (211.3, 202.0)
- added X1: ECS-2520MVLC, Oscillator:Oscillator_SMD_ECS_2520MV-xxx-xx-4Pin_2.5x2.0mm, F.Cu at (207.6, 202.0)
- added Y1: XYDBPCNANF-12MHZ, Crystal:Crystal_SMD_2520-4Pin_2.5x2.0mm, F.Cu at (222.8, 210.2)
- added Y2: XYDBPCNANF-12MHZ, Crystal:Crystal_SMD_2520-4Pin_2.5x2.0mm, F.Cu at (98.1, 224.9)
- added Y3: XYDBPCNANF-12MHZ, Crystal:Crystal_SMD_2520-4Pin_2.5x2.0mm, F.Cu at (401.9, 146.1)
- C1: value 10uF -> 0.1uF; footprint Capacitor_SMD:C_0805_2012Metric_Pad1.18x1.45mm_HandSolder -> Capacitor_SMD:C_0603_1608Metric
- C10, C13, C6, C7, C9: value 1uF -> 0.1uF; footprint Capacitor_SMD:C_0805_2012Metric_Pad1.18x1.45mm_HandSolder -> Capacitor_SMD:C_0402_1005Metric
- C11: value 22uF -> 1uF; footprint Capacitor_SMD:C_0805_2012Metric_Pad1.18x1.45mm_HandSolder -> Capacitor_SMD:C_0402_1005Metric
- C12, C36, C37, C8: footprint Capacitor_SMD:C_0805_2012Metric_Pad1.18x1.45mm_HandSolder -> Capacitor_SMD:C_0402_1005Metric
- C14, C38: value 0.1uF -> 1uF; footprint Capacitor_SMD:C_0805_2012Metric_Pad1.18x1.45mm_HandSolder -> Capacitor_SMD:C_0402_1005Metric
- C15, C16, C43: value 0.1uF -> 12pF; footprint Capacitor_SMD:C_0805_2012Metric_Pad1.18x1.45mm_HandSolder -> Capacitor_SMD:C_0402_1005Metric
- C17: value 10nF,50V -> 0.1uF,100V Tant
- C18: value 0.1uF -> 0.1uF,100V Tant
- C19, C2, C22, C23, C26, C27, C28, C3, C5, C52, C54: footprint Capacitor_SMD:C_0805_2012Metric_Pad1.18x1.45mm_HandSolder -> Capacitor_SMD:C_0603_1608Metric
- C20: value 22uF,25V -> 0.1uF; footprint Capacitor_SMD:C_0805_2012Metric_Pad1.18x1.45mm_HandSolder -> Capacitor_SMD:C_0603_1608Metric
- C21: value 0.1uF -> 10nF; footprint Capacitor_SMD:C_0805_2012Metric_Pad1.18x1.45mm_HandSolder -> Capacitor_SMD:C_0603_1608Metric
- C25: value 4.7uF,63V -> 10nF,100V; footprint Capacitor_THT:CP_Radial_D5.0mm_P2.00mm -> Capacitor_SMD:C_0805_2012Metric_Pad1.18x1.45mm_HandSolder
- C29: value 4.7uF,25V -> 30nF; footprint Capacitor_SMD:C_0805_2012Metric_Pad1.18x1.45mm_HandSolder -> Capacitor_SMD:C_0603_1608Metric
- C30, C31: value 47uF -> 0.1uF; footprint Capacitor_THT:CP_Radial_D6.3mm_P2.50mm -> Capacitor_SMD:C_0603_1608Metric
- C32: value 4.7uF,25V -> 10nF; footprint Capacitor_SMD:C_0805_2012Metric_Pad1.18x1.45mm_HandSolder -> Capacitor_SMD:C_0603_1608Metric
- C33: value 4.7uF,16V -> 0.1uF; footprint Capacitor_SMD:C_0805_2012Metric_Pad1.18x1.45mm_HandSolder -> Capacitor_SMD:C_0402_1005Metric
- C34: value 47uF -> 0.1uF; footprint Capacitor_SMD:C_1206_3216Metric_Pad1.33x1.80mm_HandSolder -> Capacitor_SMD:C_0402_1005Metric
- C39: value 2nF, 50V -> 0.1uF; footprint Capacitor_SMD:C_0805_2012Metric_Pad1.18x1.45mm_HandSolder -> Capacitor_SMD:C_0402_1005Metric
- C4, C49: value 1uF -> 0.1uF; footprint Capacitor_SMD:C_0805_2012Metric_Pad1.18x1.45mm_HandSolder -> Capacitor_SMD:C_0603_1608Metric
- C40: value 22uF,25V -> 0.1uF; footprint Capacitor_SMD:C_0805_2012Metric_Pad1.18x1.45mm_HandSolder -> Capacitor_SMD:C_0402_1005Metric
- C41: value 22uF,25V -> 1uF; footprint Capacitor_SMD:C_0805_2012Metric_Pad1.18x1.45mm_HandSolder -> Capacitor_SMD:C_0402_1005Metric
- C42: value 22uF,25V -> 12pF; footprint Capacitor_SMD:C_0805_2012Metric_Pad1.18x1.45mm_HandSolder -> Capacitor_SMD:C_0402_1005Metric
- C44, C46: value 0.1uF -> 1uF,50V
- C45, C47: value 0.1uF -> 10uF,50V
- C48: value 0.1uF -> 4.7uF,63V; footprint Capacitor_SMD:C_0805_2012Metric_Pad1.18x1.45mm_HandSolder -> Capacitor_THT:CP_Radial_D5.0mm_P2.00mm
- C58: value 0.1uF -> 4.7uF,16V Tant
- C59: value 47uF -> 1uF,16V Tant; footprint Capacitor_SMD:C_1206_3216Metric_Pad1.33x1.80mm_HandSolder -> Capacitor_SMD:C_0805_2012Metric_Pad1.18x1.45mm_HandSolder
- C65: renamed from C53; footprint Capacitor_SMD:C_0805_2012Metric_Pad1.18x1.45mm_HandSolder -> Capacitor_SMD:C_0603_1608Metric
- C69: renamed from C55; footprint Capacitor_SMD:C_0805_2012Metric_Pad1.18x1.45mm_HandSolder -> Capacitor_SMD:C_0603_1608Metric
- C71: renamed from C56; footprint Capacitor_SMD:C_0805_2012Metric_Pad1.18x1.45mm_HandSolder -> Capacitor_SMD:C_0603_1608Metric
- C73: renamed from C24; footprint Capacitor_SMD:C_0805_2012Metric_Pad1.18x1.45mm_HandSolder -> Capacitor_SMD:C_0603_1608Metric; moved to B.Cu
- C74: renamed from C51; footprint Capacitor_SMD:C_0805_2012Metric_Pad1.18x1.45mm_HandSolder -> Capacitor_SMD:C_0603_1608Metric; moved to B.Cu
- C78: renamed from C35; footprint Capacitor_SMD:C_0805_2012Metric_Pad1.18x1.45mm_HandSolder -> Capacitor_SMD:C_0603_1608Metric
- CP1: value 220uF, 50V -> 680uF,63V; footprint Capacitor_THT:CP_Radial_D12.5mm_P5.00mm -> Capacitor_THT:CP_Radial_D16.0mm_P7.50mm
- CP2: value 470uF,25V -> 680uF,63V; footprint Capacitor_THT:CP_Radial_D8.0mm_P3.50mm -> Capacitor_THT:CP_Radial_D16.0mm_P7.50mm
- CP3: value 470uF, 63V -> 470uF,63V; footprint Capacitor_THT:CP_Radial_D12.5mm_P5.00mm -> Capacitor_THT:CP_Radial_D8.0mm_P3.50mm
- CP4: value 470uF,25V -> 470uF, 63V; footprint Capacitor_THT:CP_Radial_D10.0mm_P5.00mm -> Capacitor_THT:CP_Radial_D12.5mm_P5.00mm
- CP5: value 390uF,10V -> 47uF,63V; footprint Capacitor_THT:CP_Radial_D8.0mm_P3.50mm -> Capacitor_THT:CP_Radial_D6.3mm_P2.50mm
- CP6: value 390uF,10V -> 470uF,25V; footprint Capacitor_THT:CP_Radial_D8.0mm_P3.50mm -> Capacitor_THT:CP_Radial_D10.0mm_P5.00mm
- CP7: value 470uF,25V -> 470uF,50V
- CP8: value 47uF,63V -> 22uF,63V; footprint Capacitor_THT:CP_Radial_D6.3mm_P2.50mm -> Capacitor_THT:C_Radial_D5.0mm_H11.0mm_P2.00mm
- D1: value S07G-M -> Red,150mcd; footprint Diode_SMD:D_SMF -> LED_SMD:LED_1206_3216Metric_Pad1.42x1.75mm_HandSolder
- D10, D6, D7: value B140-E3 -> Red,150mcd; footprint Diode_SMD:D_SMA -> LED_SMD:LED_1206_3216Metric_Pad1.42x1.75mm_HandSolder
- D11: value S07G-M -> B150-E3,50V; footprint Diode_SMD:D_SMF -> Diode_SMD:D_SMA
- D12: value S07G-M -> LED_CHR; footprint Diode_SMD:D_SMF -> LED_SMD:LED_0603_1608Metric
- D13: value PLZ3V6A,3.45-3.7V -> LED_CHR; footprint Diode_SMD:D_SMF -> LED_SMD:LED_0603_1608Metric
- D18: value Red,150mcd -> BAV99; footprint LED_SMD:LED_1206_3216Metric_Pad1.42x1.75mm_HandSolder -> Package_TO_SOT_SMD:SOT-23
- D19: value Red,150mcd -> SMAJ54CA; footprint LED_SMD:LED_1206_3216Metric_Pad1.42x1.75mm_HandSolder -> Diode_SMD:D_SMA
- D2: value LED -> SMAJ54CA; footprint LED_SMD:LED_0805_2012Metric_Pad1.15x1.40mm_HandSolder -> Diode_SMD:D_SMA
- D20, D21: value Orange,160mcd -> S07G-M; footprint LED_SMD:LED_1206_3216Metric_Pad1.42x1.75mm_HandSolder -> Diode_SMD:D_SMF
- D3: value B140-E3 -> SMAJ40CA; footprint Diode_SMD:D_SMA -> PCM_Diode_SMD_AKL:D_SMA
- D4, D8: value B140-E3 -> B150-E3,50V
- D5: value S07G-M -> B160-E3,60V; footprint Diode_SMD:D_SMF -> PCM_Diode_SMD_Handsoldering_AKL:D_SMB
- D9: value B140-E3 -> PLZ3V6A,3.45-3.7V; footprint Diode_SMD:D_SMA -> Diode_SMD:D_SMF
- F1, F2: footprint Fuse:Fuseholder_Cylinder-5x20mm_Schurter_0031_8201_Horizontal_Open -> Fuse:Fuse_Schurter_UMZ250
- J1: value 8-way_Screw -> SAMTEC_ET60_24S_2Pr_Pins; footprint TerminalBlock_Phoenix:TerminalBlock_Phoenix_MKDS-3-8-5.08_1x08_P5.08mm_Horizontal -> solarpump:SAMTEC_ET60T-000-3-08-D02-X-R1-S
- J11: value OLED_SOG320132A_M383 -> 3v3; footprint solarpump:OLED_SOG320132A_M383 -> TestPoint:TestPoint_Plated_Hole_D2.0mm
- J13: moved to F.Cu
- J14: value Gnd -> Fan_M; footprint TestPoint:TestPoint_Plated_Hole_D2.0mm -> Connector:FanPinHeader_1x03_P2.54mm_Vertical
- J15: value 3v3 -> USB_B_Micro; footprint TestPoint:TestPoint_Plated_Hole_D2.0mm -> Connector_USB:USB_Micro-B_Amphenol_10104110_Horizontal
- J16: value AT85_PROG -> PJ-082BH Jack Socket; footprint Connector_PinHeader_2.00mm:PinHeader_2x05_P2.00mm_Vertical -> solarpump:BarrelJack_CUI_PJ-082BH_Horizontal
- J17: value USB_B_Micro -> Amass_XT30PW; footprint Connector_USB:USB_Micro-B_Molex_47346-0001 -> solarpump:Amass_XT30PW; moved to F.Cu
- J2: value UART_IO -> SAMTEC_ET60_24S_2Pr_Socket; footprint Connector_PinHeader_2.00mm:PinHeader_1x04_P2.00mm_Vertical -> solarpump:SAMTEC_ET60S-000-3-08-D02-L-R1-S
- J3: value AUX_POWER -> SAMTEC_ET60_24S_2Pr_Socket; footprint Connector_PinHeader_2.00mm:PinHeader_1x04_P2.00mm_Vertical -> solarpump:SAMTEC_ET60S-000-3-08-D02-L-R1-S
- J4: value USB_A -> AUX_POWER; footprint solarpump:USB_Receptacle_Type_A_GCT -> Connector_PinHeader_2.00mm:PinHeader_1x04_P2.00mm_Vertical
- J5: value Conn_DISP -> UART_IO; footprint Connector_PinHeader_2.00mm:PinHeader_2x08_P2.00mm_Vertical -> Connector_PinHeader_2.00mm:PinHeader_1x04_P2.00mm_Vertical
- J8: value Flow_M -> SAMTEC_ET60_24S_2Pr_Pins; footprint Connector:FanPinHeader_1x03_P2.54mm_Vertical -> solarpump:SAMTEC_ET60T-000-3-08-D02-X-R1-S
- JP1: value AVDD_POW1 -> 10AWG; footprint Jumper:SolderJumper-2_P1.3mm_Open_RoundedPad1.0x1.5mm -> PCM_Jumper_AKL:Jumper_P5.08mm_D1.2mm
- JP2: value AVDD_POW2 -> 10AWG; footprint Jumper:SolderJumper-2_P1.3mm_Open_RoundedPad1.0x1.5mm -> PCM_Jumper_AKL:Jumper_P5.08mm_D1.2mm
- JP6: value DVDD_POW1 -> HIN_LIN; footprint Jumper:SolderJumper-2_P1.3mm_Open_RoundedPad1.0x1.5mm -> Jumper:SolderJumper-3_P1.3mm_Bridged2Bar12_RoundedPad1.0x1.5mm_NumberLabels
- L1: value 68uH -> 68uH,30A
- L2: value 68uH -> 470nH,>32A; footprint Inductor_SMD:L_12x12mm_H8mm -> Inductor_SMD:L_Chilisin_BMRF00101040
- L3: value 100uH -> 68uH; footprint Inductor_SMD:L_10.4x10.4_H4.8 -> Inductor_SMD:L_12x12mm_H8mm
- L4: value 100uH -> 22uH, 750mA
- L5: value 68uH -> 68uH,15A
- Q1: value IPP019N08NF2S -> BC817; footprint solarpump:TO-220-3_StaggeredB_Vertical -> Package_TO_SOT_SMD:SOT-23
- Q10: value Si2306BDS -> IRLB8721PBF; footprint Package_TO_SOT_SMD:SOT-23 -> Package_TO_SOT_THT:TO-220-3_Vertical
- Q2, Q3: value IPP019N08NF2S -> SQM120P10; footprint solarpump:TO-220-3_StaggeredB_Vertical -> Package_TO_SOT_SMD:TO-263-2
- Q4, Q5: value Si2306BDS -> IPP019N08NF2S; footprint Package_TO_SOT_SMD:SOT-23 -> Package_TO_SOT_THT:TO-220-3_Vertical
- Q7, Q8: value IRLB8721PBF -> IPP019N08NF2S
- R1, R4: value 4.7k -> 3K3; footprint Resistor_SMD:R_0805_2012Metric_Pad1.20x1.40mm_HandSolder -> Resistor_SMD:R_0603_1608Metric
- R10: value 10k -> 300R; footprint Resistor_SMD:R_0805_2012Metric_Pad1.20x1.40mm_HandSolder -> Resistor_SMD:R_0603_1608Metric
- R11, R34, R9: value 10k -> 10K; footprint Resistor_SMD:R_0805_2012Metric_Pad1.20x1.40mm_HandSolder -> Resistor_SMD:R_0603_1608Metric
- R12, R31: value 0R -> 10K; footprint Resistor_SMD:R_0805_2012Metric_Pad1.20x1.40mm_HandSolder -> Resistor_SMD:R_0603_1608Metric
- R13: value 0R -> 27R; footprint Resistor_SMD:R_0805_2012Metric_Pad1.20x1.40mm_HandSolder -> Resistor_SMD:R_0603_1608Metric
- R14: value 10k -> 27R; footprint Resistor_SMD:R_0805_2012Metric_Pad1.20x1.40mm_HandSolder -> Resistor_SMD:R_0603_1608Metric
- R15, R16, R37, R38: value 10k -> 100R; footprint Resistor_SMD:R_0805_2012Metric_Pad1.20x1.40mm_HandSolder -> Resistor_SMD:R_0603_1608Metric
- R17: value 22k -> 10k; footprint Resistor_SMD:R_0805_2012Metric_Pad1.20x1.40mm_HandSolder -> Resistor_SMD:R_0603_1608Metric
- R18: value 1k -> 470k; footprint Resistor_SMD:R_0805_2012Metric_Pad1.20x1.40mm_HandSolder -> Resistor_SMD:R_0603_1608Metric
- R19, R29, R30, R33: footprint Resistor_SMD:R_0805_2012Metric_Pad1.20x1.40mm_HandSolder -> Resistor_SMD:R_0603_1608Metric
- R2: value 4.7k -> 68K; footprint Resistor_SMD:R_0805_2012Metric_Pad1.20x1.40mm_HandSolder -> Resistor_SMD:R_0603_1608Metric
- R20: value 4.7k -> 1R,1W; footprint Resistor_SMD:R_0805_2012Metric_Pad1.20x1.40mm_HandSolder -> PCM_Resistor_SMD_AKL:R_2512_6332Metric
- R21: value 21.8k,0.5% -> 1R,1W; footprint Resistor_SMD:R_0805_2012Metric_Pad1.20x1.40mm_HandSolder -> PCM_Resistor_SMD_AKL:R_2512_6332Metric
- R22: value 2.5k,0.5% -> 470k; footprint Resistor_SMD:R_0805_2012Metric_Pad1.20x1.40mm_HandSolder -> Resistor_SMD:R_0603_1608Metric
- R27, R28: value 10k -> 0R; footprint Resistor_SMD:R_0805_2012Metric_Pad1.20x1.40mm_HandSolder -> Resistor_SMD:R_0603_1608Metric
- R3: value 4.7k -> 22K; footprint Resistor_SMD:R_0805_2012Metric_Pad1.20x1.40mm_HandSolder -> Resistor_SMD:R_0603_1608Metric
- R32: value 0R -> 220k; footprint Resistor_SMD:R_0805_2012Metric_Pad1.20x1.40mm_HandSolder -> Resistor_SMD:R_0603_1608Metric
- R35: value 33K,1% -> 27R; footprint Resistor_SMD:R_0805_2012Metric_Pad1.20x1.40mm_HandSolder -> Resistor_SMD:R_0603_1608Metric
- R36: value 1k -> 27R; footprint Resistor_SMD:R_0805_2012Metric_Pad1.20x1.40mm_HandSolder -> Resistor_SMD:R_0603_1608Metric
- R39, R40: value 10k -> 72R; footprint Resistor_SMD:R_0805_2012Metric_Pad1.20x1.40mm_HandSolder -> Resistor_SMD:R_0603_1608Metric
- R41: value 100R -> 21.8k,0.5%; footprint Resistor_SMD:R_0805_2012Metric_Pad1.20x1.40mm_HandSolder -> Resistor_SMD:R_0603_1608Metric
- R42: value 100R -> 2.5k,0.5%; footprint Resistor_SMD:R_0805_2012Metric_Pad1.20x1.40mm_HandSolder -> Resistor_SMD:R_0603_1608Metric
- R43: value 10k -> 4.7k; footprint Resistor_SMD:R_0805_2012Metric_Pad1.20x1.40mm_HandSolder -> Resistor_SMD:R_0603_1608Metric
- R44: value 10k -> 620R; footprint Resistor_SMD:R_0805_2012Metric_Pad1.20x1.40mm_HandSolder -> Resistor_SMD:R_0603_1608Metric
- R45: value 22k -> 100K; footprint Resistor_SMD:R_0805_2012Metric_Pad1.20x1.40mm_HandSolder -> Resistor_SMD:R_0603_1608Metric
- R46: value 1k -> 54.9K,0.5%; footprint Resistor_SMD:R_0805_2012Metric_Pad1.20x1.40mm_HandSolder -> Resistor_SMD:R_0603_1608Metric
- R5: value 6.8k -> 3K3; footprint Resistor_SMD:R_0805_2012Metric_Pad1.20x1.40mm_HandSolder -> Resistor_SMD:R_0603_1608Metric
- R50: value 10k -> 680R; footprint Resistor_SMD:R_0805_2012Metric_Pad1.20x1.40mm_HandSolder -> Resistor_SMD:R_0603_1608Metric
- R52: value 62R -> 220R; footprint Resistor_SMD:R_0805_2012Metric_Pad1.20x1.40mm_HandSolder -> Resistor_SMD:R_0603_1608Metric
- R53, R54: value 10k -> 1K; footprint Resistor_SMD:R_0805_2012Metric_Pad1.20x1.40mm_HandSolder -> Resistor_SMD:R_0603_1608Metric
- R55, R56: value 100R -> 1K; footprint Resistor_SMD:R_0805_2012Metric_Pad1.20x1.40mm_HandSolder -> Resistor_SMD:R_0603_1608Metric
- R57: value 72R -> 22K; footprint Resistor_SMD:R_0805_2012Metric_Pad1.20x1.40mm_HandSolder -> Resistor_SMD:R_0603_1608Metric
- R58: value 620R -> 22K; footprint Resistor_SMD:R_0805_2012Metric_Pad1.20x1.40mm_HandSolder -> Resistor_SMD:R_0603_1608Metric
- R59: value 160R -> 22K; footprint Resistor_SMD:R_0805_2012Metric_Pad1.20x1.40mm_HandSolder -> Resistor_SMD:R_0603_1608Metric
- R6: value 10k -> 4K7; footprint Resistor_SMD:R_0805_2012Metric_Pad1.20x1.40mm_HandSolder -> Resistor_SMD:R_0603_1608Metric
- R60: value 10k -> 22K; footprint Resistor_SMD:R_0805_2012Metric_Pad1.20x1.40mm_HandSolder -> Resistor_SMD:R_0603_1608Metric
- R61: renamed from R47; footprint Resistor_SMD:R_0805_2012Metric_Pad1.20x1.40mm_HandSolder -> Resistor_SMD:R_0603_1608Metric
- R62: renamed from R48; footprint Resistor_SMD:R_0805_2012Metric_Pad1.20x1.40mm_HandSolder -> Resistor_SMD:R_0603_1608Metric
- R63: renamed from R49; footprint Resistor_SMD:R_0805_2012Metric_Pad1.20x1.40mm_HandSolder -> Resistor_SMD:R_0603_1608Metric
- R64: renamed from R23; footprint Resistor_SMD:R_0805_2012Metric_Pad1.20x1.40mm_HandSolder -> Resistor_SMD:R_0603_1608Metric; moved to B.Cu
- R65: renamed from R24; footprint Resistor_SMD:R_0805_2012Metric_Pad1.20x1.40mm_HandSolder -> Resistor_SMD:R_0603_1608Metric; moved to B.Cu
- R69: renamed from R51; footprint Resistor_SMD:R_0805_2012Metric_Pad1.20x1.40mm_HandSolder -> Resistor_SMD:R_0603_1608Metric
- R7: value 47k -> 10K; footprint Resistor_SMD:R_0805_2012Metric_Pad1.20x1.40mm_HandSolder -> Resistor_SMD:R_0603_1608Metric
- R70: renamed from R26; footprint Resistor_SMD:R_0805_2012Metric_Pad1.20x1.40mm_HandSolder -> Resistor_SMD:R_0603_1608Metric
- R72: renamed from R25; footprint Resistor_SMD:R_0805_2012Metric_Pad1.20x1.40mm_HandSolder -> Resistor_SMD:R_0603_1608Metric
- R8: value 1k -> 4K7; footprint Resistor_SMD:R_0805_2012Metric_Pad1.20x1.40mm_HandSolder -> Resistor_SMD:R_0603_1608Metric
- SW2: value Rotary Enc EC11E -> SW_RESET; footprint solarpump:RotaryEncoder_Alps_EC11E-Switch_Vertical_H20mm_Inset_THT -> Button_Switch_SMD:SW_SPST_B3U-1000P
- SW7: value ~{BOOTSEL} -> Rotary Enc EC11E; footprint Button_Switch_SMD:SW_SPST_CK_KXT3 -> Rotary_Encoder:RotaryEncoder_Alps_EC11E-Switch_Vertical_H20mm
- U10: value MCP23017_SO -> ADS131M04-PW; footprint Package_SO:SOIC-28W_7.5x17.9mm_P1.27mm -> Package_SO:TSSOP-20_4.4x6.5mm_P0.65mm
- U12: value ACS758xCB -> SN65HVD234; footprint solarpump:Allegro_CB_PFF -> Package_SO:SOIC-8_3.9x4.9mm_P1.27mm
- U13: value ACS758xCB -> W25Q32JV; footprint solarpump:Allegro_CB_PFF -> Package_SON:WSON-8-1EP_6x5mm_P1.27mm_EP3.4x4mm
- U15: value ATtiny85-20S -> ACS71240; footprint Package_SO:SOIC-8W_5.3x5.3mm_P1.27mm -> Package_SO:SOIC-8_3.9x4.9mm_P1.27mm
- U2: value ADS130E08 -> LM386; footprint Package_QFP:TQFP-64_10x10mm_P0.5mm -> Package_SO:SOIC-8_3.9x4.9mm_P1.27mm
- U3: value ACS758xCB -> SN65HVD233; footprint solarpump:Allegro_CB_PFF -> Package_SO:SOIC-8_3.9x4.9mm_P1.27mm
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- renumbered D14 to D15, D15 to D16, D16 to D17, H8 to H10, H5 to H7, H6 to H8, H7 to H9, J12 to J25, J6 to J9, Q6 to Q9, SW1 to SW8, TP5 to TP1, U14 to U21
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Connections:
- net /FrontPanel/+3Vbat renamed /CONTROL PANEL/+3Vbat
- BT2 pad 2: /FrontPanel/FP_GND -> FPGND
- C1 pad 1: GNDA -> GND
- C1 pad 2: Net-(U2-VREF+) -> +3V3
- C10 pad 1: GND -> +3V3
- C10 pad 2: Net-(U2-VCAP3) -> GND
- C11 pad 1: GND -> +3V3
- C11 pad 2: Net-(U2-VCAP1) -> GND
- C12 pad 1: GND -> Net-(U7-VREG_VOUT)
- C12 pad 2: Net-(U2-VCAP2) -> GND
- C13 pad 1: GND -> Net-(U7-VREG_VOUT)
- C13 pad 2: Net-(U2-VCAP2) -> GND
- C14 pad 1: /MCU/VCurrent_Solr -> Net-(U7-VREG_VOUT)
- C15 pad 1: /MCU/VSolr+ -> Net-(U7-XIN)
- C15 pad 2: GNDA -> GND
- C16 pad 1: +3V3 -> Net-(U7-XOUT)
- C17 pad 1: Net-(U4-BOOT) -> Net-(D4-A)
- C17 pad 2: MPPT_Com -> /MPPT1/SOLR_RAW+
- C18 pad 1: /MPPT/SOLR_IN_M -> Net-(D4-A)
- C18 pad 2: /MPPT/BACK_gate -> /MPPT1/SOLR_LIM
- C19 pad 1: Net-(Q4-D) -> MPGND
- C19 pad 2: +12V -> MP3V3
- C2 pad 1: GNDA -> +3V3
- C2 pad 2: Net-(U2-VREF+) -> GND
- C20 pad 1: MPPT_OUT -> /MPPT1/VSolr+
- C20 pad 2: GND -> MPGND
- C21 pad 1: /MCU/VCurrent_Load -> MPGND
- C21 pad 2: GND -> /MPPT1/VCur_Solr+
- C22 pad 1: /MCU/VLoad+ -> MPGND
- C22 pad 2: GNDA -> /MPPT1/SOLR_MPPT_IN
- C23 pad 1: +3V3 -> MPGND
- C23 pad 2: GND -> MP3V3
- C25 pad 1: +BATT -> Net-(U11-BOOT)
- C25 pad 2: GND -> /MPPT1/MPPT_NODE
- C26 pad 1: Net-(U7-~{SD}/SS) -> MPGND
- C26 pad 2: GND -> Net-(U10-CAP)
- C27 pad 1: Net-(U7-Delay) -> MPGND
- C27 pad 2: GND -> MP3V3
- C28 pad 1: +12V -> MPGND
- C28 pad 2: Net-(U7-FB) -> MP3V3
- C29 pad 1: +12V -> FPGND
- C29 pad 2: GND -> Net-(C29-Pad2)
- C3 pad 1: GNDA -> GND
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Routing:
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- added copper zone on In2.Cu, net +3V3
- added copper zone on F.Cu, net +5V
- added copper zone on F.Cu, net /BATTERY/+BattPwr
- added copper zone on B.Cu, net /MPPT1/MPPT_IN
- added copper zone on F.Cu, net /MPPT1/MPPT_NODE
- added copper zone on F.Cu, net /MPPT1/MPPT_OUT
- added copper zone on F.Cu, net /MPPT1/MPPT_OUT_F
- added copper zone on F.Cu, net /MPPT1/MPPT_OUT_M
- added copper zone on F.Cu, net /MPPT1/SOLR_IV
- added copper zone on F.Cu, net /MPPT1/SOLR_LIM
- added copper zone on B.Cu, net /MPPT1/SOLR_MPPT_IN
- added copper zone on F.Cu, net /MPPT1/SOLR_MPPT_IN
- added copper zone on F.Cu, net /MPPT1/SOLR_RAW+
- added copper zone on F.Cu, net /MP_Load_P
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Other:
- board size 174.6 x 156.5 mm -> 373.1 x 220.9 mm
- copper layers 2 -> 4
- board text added: "+"
- board text added: "1"
- board text added: "12V Pwr"
- board text added: "16"
- board text added: "3V3 Pwr"
- board text added: "40"
- board text added: "BUZR"
- board text added: "CAN#1"
- board text added: "CAN#2"
- board text added: "CAN#3"
- board text added: "CAN#4"
- board text added: "Console"
- board text added: "DA/CD"
- board text added: "FAN"
- board text added: "FP#1"
- board text added: "FP#2"
- board text added: "FP#3"
- board text added: "FP#4"
- board text added: "INT SCK SI SO CS GND VCC"
- board text added: "LB"
- board text added: "LCD#1"
- board text added: "LCD#2"
- board text added: "LCD#3"
- board text added: "LCD#4"
- board text added: "PG"
- board text added: "RASPBERRY PI ZERO 2 W"
- board text added: "RPZ#1"
- board text added: "RPZ#2"
- board text added: "RPZ#3"
- board text added: "RPZ#4"
- board text added: "RPi I2C"
- board text added: "SPKR"
- board text added: "SolarPump V4 D ${REVISION} Ruth Ivimey-Cook 2021-24"
- board text added: "SwDebug"
- board text added: "TO MAIN BOARD"
- board text added: "TO SPI CANBUS MODULE"
- board text removed: "1 3V3 2 GND 3 SPICS1 4 SPIMOSI 5 SPIDC 6 SPICLK 7 SPICS2 8 GND 9 I2SCL 10 I2SDA 11 I2INT 12 GND 13 I2RST 14 3V3 15 3V3 16 GND"
- board text removed: "12V"
- board text removed: "12V 5V 3V3 GND"
- board text removed: "3V3 TX RX GND"
- board text removed: "5V"
- board text removed: "A+"
- board text removed: "BAT"
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