File: solarpump.kicad_pcb (KiCad board)
At the start: 4 copper layers, 373.1 x 220.9 mm, 450 parts, among them J1 SAMTEC_ET60_24S_2Pr_Pins, J10 SAMTEC_ET60_24S_2Pr_Socket, J11 3v3, J12 Gnd, J13 JST SM03B-SRSS-TB, J14 Fan_M, J15 USB_B_Micro, J16 PJ-082BH Jack Socket, J17 Amass_XT30PW, J18 Wire_Solr_N, J19 Wire_Solr_P, J2 SAMTEC_ET60_24S_2Pr_Socket, J20 JST SM03B-SRSS-TB, J21 JST SM03B-SRSS-TB, J22 USB_B_Micro, J23 OLED_SOG320132A_M383, J24 uHAT, J25 Stemma-QT_QWIIC, J26 JST SM03B-SRSS-TB, J27 JST SM03B-SRSS-TB, J28 USB_B_Micro, J29 OP_Wire_Aux_P, J3 SAMTEC_ET60_24S_2Pr_Socket, J30 OP_Wire_Aux_N, J31 OP_Wire_Pump_P, J32 OP_Wire_Pump_N, J33 Amass_XT30PW, J34 Amass_XT30PW, J35 Screw_Terminal_01x02, J37 Flow_M, J38 Speaker, J39 Buzzer, J4 AUX_POWER, J41 Conn_DISP, J5 UART_IO, J6 Conn_DISP, J7 SAMTEC_ET60_24S_2Pr_Pins, J8 SAMTEC_ET60_24S_2Pr_Pins, J9 Conn_DISP, M1 SPI_CAN_MOD, Q1 BC817, Q10 IRLB8721PBF, Q11 IRLB8721PBF, Q12 IRLB8721PBF, Q13 IRLB8721PBF, Q14 IRLB8721PBF, Q15 IRLB8721PBF, Q16 SQM120P10, Q17 BC817, Q18 SQM120P10, Q19 SQM120P10, Q2 SQM120P10, Q21 BC817, Q22 SQM120P10, Q23 SQM120P10, Q24 BC817, Q25 SQM120P10, Q26 SQM120P10, Q27 Si2306BDS, Q3 SQM120P10, Q4 IPP019N08NF2S, Q5 IPP019N08NF2S, Q6 IPP019N08NF2S, Q7 IPP019N08NF2S, Q8 IPP019N08NF2S, Q9 Si2306BDS, SW1 SW_RESET, SW10 SW_SPST, SW2 SW_RESET, SW3 SW_A, SW4 SW_B, SW5 SW_X, SW6 SW_Y, SW7 Rotary Enc EC11E, SW8 STOP_SW, SW9 SW_RESET, U1 AT24C040, U10 ADS131M04-PW, U11 L6398D, U12 SN65HVD234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

Commit message: pcb net updates
Parts:
- moved G*** 0.81 mm to (184.9, 44.7)
- moved R24 0.69 mm to (76.2, 214.2)
- moved C72 0.59 mm to (266.9, 46.8)
- moved R60 0.59 mm to (270.2, 46.8)
- moved R25 0.55 mm to (76.3, 217.6)
- moved R56 0.55 mm to (273.5, 46.8)
- moved C67 0.46 mm to (267.0, 55.1)
- moved R53 0.46 mm to (273.5, 55.1)
- moved R57 0.46 mm to (270.2, 55.1)
- moved C68 0.46 mm to (266.9, 52.3)
- moved C70 0.46 mm to (266.9, 49.5)
- moved R54 0.46 mm to (273.5, 52.3)
- moved R55 0.46 mm to (273.5, 49.5)
- moved R58 0.46 mm to (270.2, 52.3)
- moved R59 0.46 mm to (270.2, 49.5)
Routing:
- net (no net): track 18.8 -> 14.1 mm
- net /CONTROL PANEL/I2C_INT: track 57.3 -> 54.7 mm, vias 1 -> 2
- net /MPPT1/A1V66: track 11.7 -> 13.2 mm
- net /CONTROL PANEL/DISP_SW_A: track 66.1 -> 64.7 mm, vias 1 -> 0
- net Net-(U21-32kHz): track 11.6 -> 12.6 mm
- net Net-(SW3-B): track 35.7 -> 34.9 mm
- net /CONTROL PANEL/SPI_DC: track 65.5 -> 64.7 mm
- net Net-(SW4-B): track 42.4 -> 41.6 mm
- net Net-(SW6-B): track 58.1 -> 57.3 mm
- net /CONTROL PANEL/SPI_CS0: track 83.0 -> 82.3 mm
- net MP12V: track 48.9 -> 48.3 mm
- net FP5V: track 161.0 -> 161.6 mm, vias 5 -> 6
- net FPGND: track 70.5 -> 70.3 mm, vias 33 -> 36
- net MPGND: vias 192 -> 190
- added copper zone on F.Cu, net OP_GND
