File: misc_io.kicad_sch (KiCad schematic)
At the start: 7 parts, among them M1 Pico_Display_Pack, Q5 Si2306BDS, U11 MCP23008-xSO

Commit message: More updates to regularise property names
Parts:
- C25, C26: Manuf (none) -> KEMET; Mfr KEMET -> (none); Mfr Part No C0402C104K8R7411 -> (none); Part (none) -> C0402C104K8R7411; Supl Mouser -> (none); Supl Part No 80-C0402C104K8R7411 -> (none); Supl Price 0.016 -> (none); Vendor (none) -> Mouser; Vendor Cost (none) -> 0.016; Vendor SKU (none) -> 80-C0402C104K8R7411
- Q5: Manuf (none) -> Vishay; Mfr Vishay -> (none); Mfr Part No SI2306BDS-T1-E3 -> (none); Part (none) -> SI2306BDS-T1-E3; Supl Mouser -> (none); Supl Part No 781-SI2306BDS-E3 -> (none); Supl Price 0.496 -> (none); Vendor (none) -> Mouser; Vendor Cost (none) -> 0.496; Vendor SKU (none) -> 781-SI2306BDS-E3
Changed lines of the file:
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@@
       (effects (font (size 1.27 1.27)) hide)
     )
-    (property "Mfr" "KEMET" (id 4) (at 85.09 50.8 0)
+    (property "Manuf" "KEMET" (id 4) (at 85.09 50.8 0)
       (effects (font (size 1.27 1.27)) hide)
     )
-    (property "Mfr Part No" "C0402C104K8R7411" (id 5) (at 85.09 50.8 0)
+    (property "Part" "C0402C104K8R7411" (id 5) (at 85.09 50.8 0)
       (effects (font (size 1.27 1.27)) hide)
     )
-    (property "Supl" "Mouser" (id 6) (at 85.09 50.8 0)
+    (property "Vendor" "Mouser" (id 6) (at 85.09 50.8 0)
       (effects (font (size 1.27 1.27)) hide)
     )
-    (property "Supl Part No" "80-C0402C104K8R7411" (id 7) (at 85.09 50.8 0)
+    (property "Vendor SKU" "80-C0402C104K8R7411" (id 7) (at 85.09 50.8 0)
       (effects (font (size 1.27 1.27)) hide)
     )
-    (property "Supl Price" "0.016" (id 8) (at 85.09 50.8 0)
+    (property "Vendor Cost" "0.016" (id 8) (at 85.09 50.8 0)
       (effects (font (size 1.27 1.27)) hide)
     )
@@
       (effects (font (size 1.27 1.27)) hide)
     )
-    (property "Mfr" "KEMET" (id 4) (at 149.86 48.26 0)
+    (property "Manuf" "KEMET" (id 4) (at 149.86 48.26 0)
       (effects (font (size 1.27 1.27)) hide)
     )
-    (property "Mfr Part No" "C0402C104K8R7411" (id 5) (at 149.86 48.26 0)
+    (property "Part" "C0402C104K8R7411" (id 5) (at 149.86 48.26 0)
       (effects (font (size 1.27 1.27)) hide)
     )
-    (property "Supl" "Mouser" (id 6) (at 149.86 48.26 0)
+    (property "Vendor" "Mouser" (id 6) (at 149.86 48.26 0)
       (effects (font (size 1.27 1.27)) hide)
     )
-    (property "Supl Part No" "80-C0402C104K8R7411" (id 7) (at 149.86 48.26 0)
+    (property "Vendor SKU" "80-C0402C104K8R7411" (id 7) (at 149.86 48.26 0)
       (effects (font (size 1.27 1.27)) hide)
     )
-    (property "Supl Price" "0.016" (id 8) (at 149.86 48.26 0)
+    (property "Vendor Cost" "0.016" (id 8) (at 149.86 48.26 0)
       (effects (font (size 1.27 1.27)) hide)
     )
@@
       (effects (font (size 1.27 1.27)) (justify left) hide)
     )
-    (property "Mfr" "Vishay" (id 4) (at 102.87 134.62 0)
+    (property "Manuf" "Vishay" (id 4) (at 102.87 134.62 0)
       (effects (font (size 1.27 1.27)) hide)
     )
-    (property "Mfr Part No" "SI2306BDS-T1-E3" (id 5) (at 102.87 134.62 0)
+    (property "Part" "SI2306BDS-T1-E3" (id 5) (at 102.87 134.62 0)
       (effects (font (size 1.27 1.27)) hide)
     )
-    (property "Supl" "Mouser" (id 6) (at 102.87 134.62 0)
+    (property "Vendor" "Mouser" (id 6) (at 102.87 134.62 0)
       (effects (font (size 1.27 1.27)) hide)
     )
-    (property "Supl Part No" "781-SI2306BDS-E3" (id 7) (at 102.87 134.62 0)
+    (property "Vendor SKU" "781-SI2306BDS-E3" (id 7) (at 102.87 134.62 0)
       (effects (font (size 1.27 1.27)) hide)
     )
-    (property "Supl Price" "0.496" (id 8) (at 102.87 134.62 0)
+    (property "Vendor Cost" "0.496" (id 8) (at 102.87 134.62 0)
       (effects (font (size 1.27 1.27)) hide)
     )
