File: frontpanel.kicad_sch (KiCad schematic)
At the start: 49 parts, among them J11 OLED_SOG320132A_M383, J12 Stemma-QT_QWIIC, J16 AT85_PROG, M3 Pico_Display_Pack, Q6 Si2306BDS, SW1 STOP_SW, SW2 Rotary Enc EC11E, SW3 SW_A, SW4 SW_B, SW5 SW_X, SW6 SW_Y, U10 MCP23017_SO, U14 DS3231, U15 ATtiny85-20S

Commit message: Schematic + pcb 1.3.3
Parts:
- added D17: Green,112mcd, LED_SMD:LED_1206_3216Metric_Pad1.42x1.75mm_HandSolder, symbol Device:LED
- added R52: 62R, Resistor_SMD:R_0805_2012Metric_Pad1.20x1.40mm_HandSolder, symbol Device:R_Small
- D14: value Orange,112mcd -> Orange,160mcd; Manuf Dialight -> Kingbright; Part 599-0230-007F -> APT3216SECK; Vendor Cost 0.33 -> 0.176; Vendor SKU 645-599-0230-007F -> 604-APT3216SECK
- D15: value Green,100mcd -> Green,112mcd; Manuf Kingbright -> Dialight; Part APTL3216CGCK-01 -> 599-0230-007F; Vendor Cost 0.30 -> 0.304; Vendor SKU 604-APTL3216CGCK-01 -> 645-599-0230-007F
- D16: value Red,100mcd -> Red,150mcd; Part APT3216SRCPRV -> APT3216SURCK; Vendor Cost 0.26 -> 0.24; Vendor SKU 604-APT3216SRCPRV -> 604-APT3216SURCK; Vf 1.85 -> 1.95
- J16: footprint Connector_PinHeader_2.00mm:PinHeader_2x03_P2.00mm_Vertical -> Connector_PinHeader_2.00mm:PinHeader_2x05_P2.00mm_Vertical; symbol Connector:Conn_01x06_Male -> Connector:Conn_01x10_Pin
- M3: footprint Package_DIP:DIP-40_W15.24mm_Socket -> solarpump:DIP-40_W17.78mm_Socket; now not fitted
- R47: Vendor Cost 0.077 -> 0.08
- R48: value 60R -> 62R; Manuf Vishay / Dale -> Yageo; Part CRCW080562R0JNEA -> AC0805FR-0762RL; Vendor Cost 0.077 -> 0.08; Vendor SKU 71-CRCW080562R0JNEA -> 603-AC0805FR-0762RL
- SW2: footprint solarpump:RotaryEncoder_Alps_EC11E-Switch_Vertical_H20mm_Inset -> solarpump:RotaryEncoder_Alps_EC11E-Switch_Vertical_H20mm_Inset_THT
- TP6: value AT85_TP -> AT85_INT
Connections:
- net FP_3V3: now also J16.2 (Pin_2), R52.1
- net FP_GND: now also C38.2, J16.9 (Pin_9); no longer C38.1
- net I2C_SCL: now also J16.4 (Pin_4); no longer J16.2 (Pin_2)
- net I2C_SDA: now also J16.8 (Pin_8); no longer J16.6 (Pin_6)
- net MISO_SW: now also J16.5 (Pin_5); no longer J16.3 (Pin_3)
- net MOSI_SDA: now also J16.7 (Pin_7); no longer J16.5 (Pin_5)
- net SCK_SCL: now also J16.3 (Pin_3); no longer J16.1 (Pin_1)
- net AT85_RES renamed RES_INT
- net RES_INT: now also J16.1 (Pin_1)
- net ROT_SW renamed SW
- net SW: now also C38.1, J16.6 (Pin_6), D17.1 (K); no longer C38.2, J16.4 (Pin_4)
- new net: D17.2 (A), R52.2
Other:
- note added: ""Alarm" Buzzer"
- note added: ""Emergency Stop" Momentary Pushbutton, red top."
- note added: "ATTINY MCU interfaces encoder to behave as an I2C device."
- note added: "Encoder has momentary short-travel push-to-make SW."
- note added: "Opt MCU monitor"
- note added: "Pico Display Pack 4 switches, 1 RGB LED 1.14" 240x135 IPS LCD 40-pin DIP (0.7" spacing)"
- note added: "Programming connector intercepts pins of MCU to enable programming"
- note added: "Rotary Encoder as UI selector with MCU interface to I2C"
- note removed: ""Emergency Stop" Momentary Pushbutton, red top. "Alarm" Buzzer"
- note removed: "Pico Display Pack 4 switches, 1 RGB LED 1.14" 240x135 IPS LCD 40-pin DIP"
- note removed: "Rotary Encoder used as UI selector, with integral SW."
- moved on the sheet: BZ1, C35, C36, C37, C38, C52, C53, C54, C55, C56, Q6, R25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

Commit message: Further works...
Parts:
- removed C36, C37, C38, C52: 0.1uF, Capacitor_SMD:C_0805_2012Metric_Pad1.18x1.45mm_HandSolder, symbol Device:C_Small
- removed D17: Green,112mcd, LED_SMD:LED_1206_3216Metric_Pad1.42x1.75mm_HandSolder, symbol Device:LED
- removed J16: AT85_PROG, Connector_PinHeader_2.00mm:PinHeader_2x05_P2.00mm_Vertical, symbol Connector:Conn_01x10_Pin
- removed M3: Pico_Display_Pack, solarpump:DIP-40_W17.78mm_Socket, symbol solarpump:Pico_Display_Pack
- removed R27, R28, R29, R50: 10k, Resistor_SMD:R_0805_2012Metric_Pad1.20x1.40mm_HandSolder, symbol Device:R_Small
- removed R52: 62R, Resistor_SMD:R_0805_2012Metric_Pad1.20x1.40mm_HandSolder, symbol Device:R_Small
- removed SW2: Rotary Enc EC11E, solarpump:RotaryEncoder_Alps_EC11E-Switch_Vertical_H20mm_Inset_THT, symbol Device:Rotary_Encoder_Switch
- removed TP3: GBP1_TP, TestPoint:TestPoint_Pad_1.0x1.0mm, symbol Connector:TestPoint
- removed TP4: GBP2_TP, TestPoint:TestPoint_Pad_1.0x1.0mm, symbol Connector:TestPoint
- removed TP6: AT85_INT, TestPoint:TestPoint_Pad_1.0x1.0mm, symbol Connector:TestPoint
- removed U10: MCP23017_SO, Package_SO:SOIC-28W_7.5x17.9mm_P1.27mm, symbol Interface_Expansion:MCP23017_SO
- removed U15: ATtiny85-20S, Package_SO:SOIC-8W_5.3x5.3mm_P1.27mm, symbol MCU_Microchip_ATtiny:ATtiny85-20S
- added C117, C120, C61: 10uF, Capacitor_SMD:C_0603_1608Metric, symbol Device:C_Small
- added C118, C67, C68, C70, C72, C75, C76, C77: 0.1uF, Capacitor_SMD:C_0603_1608Metric, symbol Device:C_Small
- added C119: 100uF, Capacitor_SMD:C_0603_1608Metric, symbol Device:C_Small
- added C29: 30nF, Capacitor_SMD:C_0603_1608Metric, symbol Device:C_Small
- added D18: BAV99, Package_TO_SOT_SMD:SOT-23, symbol Diode:BAV99
- added J24: uHAT, Module:Raspberry_Pi_Zero_Socketed_THT_FaceDown_MountingHoles, symbol Connector_Generic:Conn_02x20_Odd_Even
- added J38: Speaker, Connector_JST:JST_PH_S2B-PH-K_1x02_P2.00mm_Horizontal, symbol Connector_Generic:Conn_01x02
- added J39: Buzzer, Connector_JST:JST_PH_S2B-PH-K_1x02_P2.00mm_Horizontal, symbol Connector_Generic:Conn_01x02
- added M1: SPI_CAN_MOD, IvimeyCom:MCP2515 CAN module_SMD, symbol solarpump:SPI_CAN_MOD
- added R104: 270R, Resistor_SMD:R_0603_1608Metric, symbol Device:R_Small
- added R119: 10K, Resistor_SMD:R_0603_1608Metric, symbol Device:R_Small
- added R120: 10R, Resistor_SMD:R_0603_1608Metric, symbol Device:R_Small
- added R5: 3K3, Resistor_SMD:R_0603_1608Metric, symbol Device:R_Small
- added R53, R54, R55, R56: 1K, Resistor_SMD:R_0603_1608Metric, symbol Device:R_Small
- added R57, R58, R59, R60: 22K, Resistor_SMD:R_0603_1608Metric, symbol Device:R_Small
- added R66, R67, R68: 10k, Resistor_SMD:R_0603_1608Metric, symbol Device:R_Small
- added R71: 150R, Resistor_SMD:R_0603_1608Metric, symbol Device:R_Small
- added RV1, RV2: 10K, Potentiometer_SMD:Potentiometer_Bourns_TC33X_Vertical, symbol Device:R_Potentiometer_Trim
- added SW7: Rotary Enc EC11E, Rotary_Encoder:RotaryEncoder_Alps_EC11E-Switch_Vertical_H20mm, symbol Device:Rotary_Encoder_Switch
- added TVS5, TVS6, TVS7: TVS, Package_TO_SOT_SMD:SOT-23, symbol Diode:PESD2IVN48T
- added U2: LM386, Package_SO:SOIC-8_3.9x4.9mm_P1.27mm, symbol Amplifier_Audio:LM386
- BZ1: now not fitted; now left out of the parts list
- C65: renamed from C53; footprint Capacitor_SMD:C_0805_2012Metric_Pad1.18x1.45mm_HandSolder -> Capacitor_SMD:C_0603_1608Metric
- C66: renamed from C54; footprint Capacitor_SMD:C_0805_2012Metric_Pad1.18x1.45mm_HandSolder -> Capacitor_SMD:C_0603_1608Metric
- C69: renamed from C55; footprint Capacitor_SMD:C_0805_2012Metric_Pad1.18x1.45mm_HandSolder -> Capacitor_SMD:C_0603_1608Metric
- C71: renamed from C56; footprint Capacitor_SMD:C_0805_2012Metric_Pad1.18x1.45mm_HandSolder -> Capacitor_SMD:C_0603_1608Metric
- C73: renamed from C24; footprint Capacitor_SMD:C_0805_2012Metric_Pad1.18x1.45mm_HandSolder -> Capacitor_SMD:C_0603_1608Metric
- C74: renamed from C51; footprint Capacitor_SMD:C_0805_2012Metric_Pad1.18x1.45mm_HandSolder -> Capacitor_SMD:C_0603_1608Metric
- C78: renamed from C35; footprint Capacitor_SMD:C_0805_2012Metric_Pad1.18x1.45mm_HandSolder -> Capacitor_SMD:C_0603_1608Metric
- R61: renamed from R47; footprint Resistor_SMD:R_0805_2012Metric_Pad1.20x1.40mm_HandSolder -> Resistor_SMD:R_0603_1608Metric
- R62: renamed from R48; footprint Resistor_SMD:R_0805_2012Metric_Pad1.20x1.40mm_HandSolder -> Resistor_SMD:R_0603_1608Metric
- R63: renamed from R49; footprint Resistor_SMD:R_0805_2012Metric_Pad1.20x1.40mm_HandSolder -> Resistor_SMD:R_0603_1608Metric
- R64: renamed from R23; footprint Resistor_SMD:R_0805_2012Metric_Pad1.20x1.40mm_HandSolder -> Resistor_SMD:R_0603_1608Metric
- R65: renamed from R24; footprint Resistor_SMD:R_0805_2012Metric_Pad1.20x1.40mm_HandSolder -> Resistor_SMD:R_0603_1608Metric
- R69: renamed from R51; footprint Resistor_SMD:R_0805_2012Metric_Pad1.20x1.40mm_HandSolder -> Resistor_SMD:R_0603_1608Metric
- R70: renamed from R26; footprint Resistor_SMD:R_0805_2012Metric_Pad1.20x1.40mm_HandSolder -> Resistor_SMD:R_0603_1608Metric
- R72: renamed from R25; footprint Resistor_SMD:R_0805_2012Metric_Pad1.20x1.40mm_HandSolder -> Resistor_SMD:R_0603_1608Metric
- renumbered D14 to D15, D15 to D16, D16 to D17, J11 to J23, J12 to J25, Q6 to Q9, SW1 to SW8, TP5 to TP1, U14 to U21
Connections:
- net FP_GND is gone; now on net FPGND: BT2.2 (-), C65.2, C66.1, C69.1, C71.2, C73.1, C74.1, C78.1, D15.1 (K), D16.1 (K), D17.1 (K), J23.1 (GND), J25.4 (GND), Q9.2 (S), R69.2, R70.2, U21.10 (GND), U21.11 (GND), U21.12 (GND), U21.13 (GND), U21.5 (GND), U21.6 (GND), U21.7 (GND), U21.8 (GND), U21.9 (GND)
- net BUZZER: now also J24.40 (Pin_40)
- net DISP_LED_B: now also J24.13 (Pin_13)
- net DISP_LED_G: now also J24.15 (Pin_15)
- net DISP_LED_R: now also J24.29 (Pin_29)
- net DISP_SW_A: now also C67.1, J24.31 (Pin_31), R57.1; no longer SW3.2 (B)
- net DISP_SW_B: now also C68.1, J24.33 (Pin_33), R58.1; no longer SW4.2 (B)
- net DISP_SW_X: now also C70.1, J24.35 (Pin_35), R59.1; no longer SW5.2 (B)
- net DISP_SW_Y: now also C72.1, J24.37 (Pin_37), R60.1; no longer SW6.2 (B)
- net I2C_INT: now also J24.11 (Pin_11), M1.1 (INT); no longer U21.3 (~{INT}/SQW)
- net I2C_SCL: now also R64.2, J24.5 (Pin_5); no longer R65.2
- net I2C_SDA: now also R65.2, J24.3 (Pin_3); no longer R64.2
- net SPI_CLK: now also J24.23 (Pin_23), M1.2 (SCK)
- net SPI_CS1: now also J24.24 (Pin_24)
- net SPI_CS2: now also J24.36 (Pin_36)
- net SPI_DC: now also J24.22 (Pin_22)
- net SPI_MOSI: now also J24.19 (Pin_19), M1.3 (SI)
- net STOP_SW: now also J24.38 (Pin_38)
- net ~{RESET}: no longer U21.4 (~{RST})
- net FPGND: now reaches SW3.1 (A), SW4.1 (A), SW5.1 (A), SW6.1 (A)
- net FPGND: now also C117.1, C29.1, C67.2, C68.2, C70.2, C72.2, C75.2, C76.2, C77.2, D18.1 (K), J24.14 (Pin_14), J24.20 (Pin_20), J24.25 (Pin_25), J24.30 (Pin_30), J24.34 (Pin_34), J24.39 (Pin_39), J24.6 (Pin_6), J24.9 (Pin_9), J38.2 (Pin_2), M1.6 (GND), R120.1, R5.2, R71.2, RV1.3, SW7.C, SW7.MP, SW7.S2, TVS5.3 (common), TVS6.3 (common), TVS7.3 (common), U2.2 (-), U2.4 (GND)
- net at Q9.3 (D): now also J39.1 (Pin_1); no longer BZ1.2 (+)
- net FP_3V3 renamed FP3V3
- net FP3V3: now also D18.2 (A), J24.1 (Pin_1), J24.17 (Pin_17), M1.7 (VCC), R53.2, R54.2, R55.2, R56.2, R66.1, R67.1, R68.1; no longer BZ1.1 (-)
- new net: C120.1, RV2.2
- new net: C120.2, U2.8 (GAIN)
- new net: R53.1, R57.2, SW3.2 (B)
- new net: C118.2, R120.2
- new net: C61.1, D18.3 (K), RV1.1
- new net: C29.2, C61.2, R104.2, R71.1
- new net: R56.1, R60.2, SW6.2 (B)
- new net: C118.1, C119.1, U2.5
- new net: C119.2, J38.1 (Pin_1)
- new net: RV2.1, U2.1 (GAIN)
- new net: R119.1, U2.7 (BYPASS)
- new net: C117.2, R119.2
- new net: R55.1, R59.2, SW5.2 (B)
- new net: R54.1, R58.2, SW4.2 (B)
- new net: RV1.2, U2.3 (+)
- new net AT_ROTA: C75.1, J24.27 (Pin_27), R66.2, SW7.B
- new net AT_ROTB: C76.1, J24.28 (Pin_28), R67.2, SW7.A
- new net AT_SW: C77.1, J24.7 (Pin_7), R68.2, SW7.S1
- new net FP5V: J24.2 (Pin_2), J24.4 (Pin_4), J39.2 (Pin_2), U2.6 (V+)
- new net FP_CAN.H: M1.C2 (CAN_H), TVS5.2 (A2)
- new net FP_CAN.L: M1.C1 (CAN_L), TVS5.1 (A1)
- new net FP_MOD.~{ALARM}: J24.16 (Pin_16), TVS6.1 (A1)
- new net FP_MOD.~{RESET}: J24.18 (Pin_18), TVS6.2 (A2), U21.4 (~{RST})
- new net FP_MOD.~{SNS4}: R5.1
- new net FP_UART.RX: J24.8 (Pin_8), TVS7.1 (A1)
- new net FP_UART.TX: J24.10 (Pin_10), TVS7.2 (A2)
- new net GPIO12/PWM0: J24.32 (Pin_32)
- new net PWM0_SPKR: J24.12 (Pin_12), R104.1
- new net SPI_CS0: J24.26 (Pin_26), M1.5 (CS)
- new net SPI_MISO: J24.21 (Pin_21), M1.4 (SO)
- no-connect marks 4 -> 9
Other:
- note added: "(bypass, opt)"
- note added: "1ch Speaker output (clone of RPi circuit)"
- note added: "Connection to Raspberry Pi Zero via uHAT connector for UI / display and high level control. Main connection via CAN bus."
- note added: "Connector for Surenoo 200dpi 320x132 OLED"
- note added: "LEDs, Switches for UI"
- note added: "UI / R-PI Zero W interface"
- note added: "circuits-diy.com"
- note added: "https://www.circuits-diy.com/wp-content/uploads/2022/12/lm386-audio-amplifier-circuit-diagram-schematic.png"
- note removed: "ATTINY MCU interfaces encoder to behave as an I2C device."
- note removed: "Connector for Surenoo 200dpi 320x132 OLED (replaces Pico Display)"
- note removed: "Encoder has momentary short-travel push-to-make SW."
- note removed: "Opt MCU monitor"
- note removed: "Pico Display Pack 4 switches, 1 RGB LED 1.14" 240x135 IPS LCD 40-pin DIP (0.7" spacing)"
- note removed: "Programming connector intercepts pins of MCU to enable programming"
- note removed: "Rotary Encoder as UI selector with MCU interface to I2C"
- title: SolarPump v3 -> SolarPump v4
- moved on the sheet: BT2, C65, C66, C69, C71, C73, C74, C78, D15, D16, D17, J23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
