File: mppt.kicad_sch (KiCad schematic)
At the start: 48 parts, among them J10 Fan_F, J9 Fan_M, M1 Fan_3pin, Q1 IPP019N08NF2S, Q2 IPP019N08NF2S, Q3 IPP019N08NF2S, Q4 Si2306BDS, Q5 Si2306BDS, U3 ACS758xCB, U4 L6398D, U5 TME 1212S, U6 ACS758xCB

Commit message: Schematic + pcb 1.3.3
Parts:
- HS1, HS2, HS3: value Heatsink -> HSink
- R12, R13: value 0 -> 0R

Commit message: Further works...
Parts:
- removed C21: 0.1uF, Capacitor_SMD:C_0805_2012Metric_Pad1.18x1.45mm_HandSolder, symbol Device:C_Small
- removed D1, D5: S07G-M, Diode_SMD:D_SMF, symbol Diode:1N4007
- removed D2: LED, LED_SMD:LED_0805_2012Metric_Pad1.15x1.40mm_HandSolder, symbol Device:LED
- removed D3: B140-E3, Diode_SMD:D_SMA, symbol Device:D_Schottky
- removed HS3: HSink, MountingHole:MountingHole_2.7mm_M2.5_Pad_Via, symbol Mechanical:Heatsink_Pad
- removed J10: Fan_F, symbol Connector:Conn_01x03_Male
- removed J9: Fan_M, Connector:FanPinHeader_1x03_P2.54mm_Vertical, symbol Connector:Conn_01x03_Female
- removed M1: Fan_3pin, symbol Motor:Fan_3pin
- removed Q4, Q5: Si2306BDS, Package_TO_SOT_SMD:SOT-23, symbol solarpump:Si2306BDS
- removed R10, R11, R16: 10k, Resistor_SMD:R_0805_2012Metric_Pad1.20x1.40mm_HandSolder, symbol Device:R_Small
- removed U3, U6: ACS758xCB, solarpump:Allegro_CB_PFF, symbol Sensor_Current:ACS758xCB-050B-PFF
- removed U5: TME 1212S, solarpump:TME-1212S, symbol solarpump:ITB1212S
- added C17: 0.1uF,100V Tant, Capacitor_SMD:C_0805_2012Metric_Pad1.18x1.45mm_HandSolder, symbol Device:C_Small
- added C24, C26, C27, C28, C30: 0.1uF, Capacitor_SMD:C_0603_1608Metric, symbol Device:C_Small
- added C32: 10nF, Capacitor_SMD:C_0603_1608Metric, symbol Device:C_Small
- added C33, C34, C35, C36, C37, C39, C40: 0.1uF, Capacitor_SMD:C_0402_1005Metric, symbol Device:C_Small
- added C38, C41: 1uF, Capacitor_SMD:C_0402_1005Metric, symbol Device:C_Small
- added C42, C43: 12pF, Capacitor_SMD:C_0402_1005Metric, symbol Device:C_Small
- added C44, C46: 1uF,50V, Capacitor_SMD:C_0805_2012Metric_Pad1.18x1.45mm_HandSolder, symbol Device:C_Small
- added C45, C47: 10uF,50V, Capacitor_SMD:C_0805_2012Metric_Pad1.18x1.45mm_HandSolder, symbol Device:C_Small
- added CP2: 680uF,63V, Capacitor_THT:CP_Radial_D16.0mm_P7.50mm, symbol Device:C_Polarized_Small
- added D2: SMAJ54CA, Diode_SMD:D_SMA, symbol Diode:SMAJ54CA
- added D3: SMAJ40CA, PCM_Diode_SMD_AKL:D_SMA, symbol PCM_Diode_TVS_AKL:SMAJ40CA
- added D5: B160-E3,60V, PCM_Diode_SMD_Handsoldering_AKL:D_SMB, symbol PCM_Diode_Schottky_AKL:B160
- added D6, D7: Red,150mcd, LED_SMD:LED_1206_3216Metric_Pad1.42x1.75mm_HandSolder, symbol Device:LED
- added DZ1: BZV90-C30, Package_TO_SOT_SMD:SOT-223-3_TabPin2, symbol PCM_Diode_Zener_AKL:BZV90-C30
- added J16: PJ-082BH Jack Socket, solarpump:BarrelJack_CUI_PJ-082BH_Horizontal, symbol Connector:Barrel_Jack
- added J17: Amass_XT30PW, solarpump:Amass_XT30PW, symbol solarpump:Amass_XT30PW
- added J18: Wire_Solr_N, Connector_Wire:SolderWire-2sqmm_1x01_D2mm_OD3.9mm, symbol Connector:Conn_01x01_Socket
- added J19: Wire_Solr_P, Connector_Wire:SolderWire-2sqmm_1x01_D2mm_OD3.9mm, symbol Connector:Conn_01x01_Socket
- added J20, J21: JST SM03B-SRSS-TB, Connector_JST:JST_SH_SM03B-SRSS-TB_1x03-1MP_P1.00mm_Horizontal, symbol Connector_Generic_MountingPin:Conn_01x03_MountingPin
- added J22: USB_B_Micro, Connector_USB:USB_Micro-B_Amphenol_10104110_Horizontal, symbol Connector:USB_B_Micro
- added JP1, JP2: 10AWG, PCM_Jumper_AKL:Jumper_P5.08mm_D1.2mm, symbol Jumper:Jumper_2_Bridged
- added L2: 470nH,>32A, Inductor_SMD:L_Chilisin_BMRF00101040, symbol Device:L_Ferrite
- added Q1: BC817, Package_TO_SOT_SMD:SOT-23, symbol Transistor_BJT:BC817
- added Q2, Q3: SQM120P10, Package_TO_SOT_SMD:TO-263-2, symbol Transistor_FET:SQM120P10
- added Q7, Q8: IPP019N08NF2S, Package_TO_SOT_THT:TO-220-3_Vertical, symbol solarpump:IPP019N08NF2S
- added R17: 10k, Resistor_SMD:R_0603_1608Metric, symbol Device:R_Small
- added R18: 470k, Resistor_SMD:R_0603_1608Metric, symbol Device:R_Small
- added R20, R21: 1R,1W, PCM_Resistor_SMD_AKL:R_2512_6332Metric, symbol Device:R_Small
- added R24, R25: 4.7k,0.5%, Resistor_SMD:R_0603_1608Metric, symbol Device:R_Small
- added R31, R34: 10K, Resistor_SMD:R_0603_1608Metric, symbol Device:R_Small
- added R35, R36: 27R, Resistor_SMD:R_0603_1608Metric, symbol Device:R_Small
- added R37, R38: 100R, Resistor_SMD:R_0603_1608Metric, symbol Device:R_Small
- added R39, R40: 72R, Resistor_SMD:R_0603_1608Metric, symbol Device:R_Small
- added SW2: SW_RESET, Button_Switch_SMD:SW_SPST_B3U-1000P, symbol Switch:SW_SPST
- added TVS1, TVS2, TVS3, TVS4: TVS, Package_TO_SOT_SMD:SOT-23, symbol Diode:PESD2IVN48T
- added U10: ADS131M04-PW, Package_SO:TSSOP-20_4.4x6.5mm_P0.65mm, symbol solarpump:ADS131M04-PW
- added U12: SN65HVD234, Package_SO:SOIC-8_3.9x4.9mm_P1.27mm, symbol Interface_CAN_LIN:SN65HVD233
- added U13: W25Q32JV, Package_SON:WSON-8-1EP_6x5mm_P1.27mm_EP3.4x4mm, symbol Memory_Flash_Extra:W25Q64JV
- added U14: RP2040, Package_DFN_QFN:QFN-56-1EP_7x7mm_P0.4mm_EP3.2x3.2mm_ThermalVias, symbol solarpump:RP2040
- added U15, U8: ACS71240, Package_SO:SOIC-8_3.9x4.9mm_P1.27mm, symbol Sensor_Current:ACS71240LLCBTR-025B3
- added U9: MAX16171, solarpump:TDFN-8-1EP_3x2mm_P0.5mm_EP1.5x1.75mm, symbol solarpump:MAX16171
- added Y2: XYDBPCNANF-12MHZ, Crystal:Crystal_SMD_2520-4Pin_2.5x2.0mm, symbol Device:Crystal_GND24_Small
- C18: value 0.1uF -> 0.1uF,100V Tant
- C19: renamed from C16; footprint Capacitor_SMD:C_0805_2012Metric_Pad1.18x1.45mm_HandSolder -> Capacitor_SMD:C_0603_1608Metric
- C20: renamed from C15; footprint Capacitor_SMD:C_0805_2012Metric_Pad1.18x1.45mm_HandSolder -> Capacitor_SMD:C_0603_1608Metric
- C21: renamed from C14; value 0.1uF -> 10nF; footprint Capacitor_SMD:C_0805_2012Metric_Pad1.18x1.45mm_HandSolder -> Capacitor_SMD:C_0603_1608Metric
- C22: renamed from C19; footprint Capacitor_SMD:C_0805_2012Metric_Pad1.18x1.45mm_HandSolder -> Capacitor_SMD:C_0603_1608Metric
- C23: footprint Capacitor_SMD:C_0805_2012Metric_Pad1.18x1.45mm_HandSolder -> Capacitor_SMD:C_0603_1608Metric; Vendor Cost 0.016 -> 0.027
- C25: renamed from C17; value 10nF,50V -> 10nF,100V
- C31: renamed from C22; footprint Capacitor_SMD:C_0805_2012Metric_Pad1.18x1.45mm_HandSolder -> Capacitor_SMD:C_0603_1608Metric
- CP1: value 220uF, 50V -> 680uF,63V; footprint Capacitor_THT:CP_Radial_D12.5mm_P5.00mm -> Capacitor_THT:CP_Radial_D16.0mm_P7.50mm; Part UPM1H221MHD6TO -> UPM1J271MHD6; Vendor SKU 647-UPM1H221MHD6TO -> 647-UPM1J271MHD6
- CP3: renamed from CP2; value 470uF,25V -> 470uF,63V
- CP8: renamed from C20; value 22uF,25V -> 22uF,63V; footprint Capacitor_SMD:C_0805_2012Metric_Pad1.18x1.45mm_HandSolder -> Capacitor_THT:C_Radial_D5.0mm_H11.0mm_P2.00mm; symbol Device:C_Small -> Device:C_Polarized_Small; Manuf Samsung Electro-Mechanics -> Rubycon; Part CL21A226MAQNNNE -> 63YXJ22M5X11; Vendor Cost 0.25 -> 0.19; Vendor SKU 187-CL21A226MAQNNNE -> 232-63YXJ22M5X11
- D4: value B140-E3 -> B150-E3,50V; DNF DNF -> (none); Part B140-E3/5AT -> B150-E3/5AT; Vendor SKU 625-B140-E3 -> 625-B150-E3
- F1, F2: footprint Fuse:Fuseholder_Cylinder-5x20mm_Schurter_0031_8201_Horizontal_Open -> Fuse:Fuse_Schurter_UMZ250
- L1: value 68uH -> 68uH,30A
- Q4: renamed from Q1; footprint solarpump:TO-220-3_StaggeredB_Vertical -> Package_TO_SOT_THT:TO-220-3_Vertical
- Q5: renamed from Q2; footprint solarpump:TO-220-3_StaggeredB_Vertical -> Package_TO_SOT_THT:TO-220-3_Vertical
- Q6: renamed from Q3; footprint solarpump:TO-220-3_StaggeredB_Vertical -> Package_TO_SOT_THT:TO-220-3_Vertical
- R19: footprint Resistor_SMD:R_0805_2012Metric_Pad1.20x1.40mm_HandSolder -> Resistor_SMD:R_0603_1608Metric
- R22: renamed from R7; value 47k -> 470k; footprint Resistor_SMD:R_0805_2012Metric_Pad1.20x1.40mm_HandSolder -> Resistor_SMD:R_0603_1608Metric
- R23: renamed from R8; value 1k -> 10k; footprint Resistor_SMD:R_0805_2012Metric_Pad1.20x1.40mm_HandSolder -> Resistor_SMD:R_0603_1608Metric
- R26: renamed from R9; footprint Resistor_SMD:R_0805_2012Metric_Pad1.20x1.40mm_HandSolder -> Resistor_SMD:R_0603_1608Metric
- R27: renamed from R12; footprint Resistor_SMD:R_0805_2012Metric_Pad1.20x1.40mm_HandSolder -> Resistor_SMD:R_0603_1608Metric
- R28: renamed from R13; footprint Resistor_SMD:R_0805_2012Metric_Pad1.20x1.40mm_HandSolder -> Resistor_SMD:R_0603_1608Metric
- R29: renamed from R14; footprint Resistor_SMD:R_0805_2012Metric_Pad1.20x1.40mm_HandSolder -> Resistor_SMD:R_0603_1608Metric
- R30: renamed from R15; footprint Resistor_SMD:R_0805_2012Metric_Pad1.20x1.40mm_HandSolder -> Resistor_SMD:R_0603_1608Metric
- R32: renamed from R17; value 22k -> 220k; footprint Resistor_SMD:R_0805_2012Metric_Pad1.20x1.40mm_HandSolder -> Resistor_SMD:R_0603_1608Metric
- R33: renamed from R18; value 1k -> 10k; footprint Resistor_SMD:R_0805_2012Metric_Pad1.20x1.40mm_HandSolder -> Resistor_SMD:R_0603_1608Metric
- renumbered U4 to U11
Connections:
- net +3V3 is gone; now on net MPGND: C19.1, C23.1
- net GNDA is gone; now on net MPGND: C20.2, C31.2
- net VCurrent_Solr+ is gone; now on net MPGND: C21.1
- net Load_P: now also F2.1; no longer F2.2
- net MPPT_BACKen: now also U14.8 (GPIO6), U9.4 (EN)
- net MPPT_Hvg: now also Q5.1 (G), R27.1, R29.1, Q7.1 (G); no longer R27.2, U11.7 (HVG)
- net MPPT_IN: now also JP2.2 (B), Q7.2 (D); no longer Q4.2 (D)
- net MPPT_Lvg: now also Q6.1 (G), R28.1, R30.1, Q8.1 (G); no longer D4.1 (K), R28.2, U11.5 (LVG)
- net MPPT_OUT: now also U15.1 (IP+), U15.2 (IP+)
- net MPPT_OUT_M: now also C44.1, C45.1, L2.1, U15.3 (IP-), U15.4 (IP-); no longer F2.1
- net MPPT_PWMhi: now also U14.11 (GPIO8)
- net MPPT_PWMlo: now also U14.12 (GPIO9)
- net VLoad+: now also U10.7 (Ain3+)
- net VSolr+: now also U10.3 (Ain1+)
- net MPGND: now reaches C22.1
- net MPGND: now also CP1.2, CP3.2, CP8.2, HS1.1, HS2.1, Q6.3 (S), R23.2, R26.2, R30.2, R33.2, U11.4 (GND), C24.1, C26.1, C27.1, C28.1, C30.1, C32.1, C33.2, C34.2, C35.2, C36.2, C37.2, C38.2, C39.2, C40.2, C41.2, C42.2, C43.2, C44.2, C45.2, C46.2, C47.2, CP2.2, D2.1 (A1), D3.1 (K), J16.2, J17.2 (Pin_2), J18.1 (Pin_1), J20.2 (Pin_2), J20.MP (MountPin), J21.1 (Pin_1), J21.MP (MountPin), J22.5 (GND), J22.6 (Shield), Q8.3 (S), R17.2, R20.2, R25.2, SW2.1 (A), TVS1.3 (common), TVS2.3 (common), TVS3.3 (common), TVS4.3 (common), U10.19 (DGND), U10.2 (AGND), U12.2 (GND), U13.4 (GND), U13.9 (GND), U14.19 (TESTEN), U14.57 (GND), U15.5 (GND), U8.5 (GND), U9.5 (GND), U9.9 (EP), Y2.2, Y2.4
- net +12V renamed MP12V
- net MP12V: no longer C22.2
- net BACK_gate: no longer names the net of Q4.1 (G)
- net BACK_gate: now also U9.1 (GATE); no longer C18.2
- net Fan_En+ renamed SOLR_INPen
- net SOLR_INPen: now also U14.9 (GPIO7)
- removed net GND: C19.2, C21.2, C23.2, CP1.2, CP3.2, CP8.2, HS1.1, HS2.1, Q6.3 (S), R19.2, R23.2, R26.2, R30.2, R33.2, U11.4 (GND)
- net MPPT_Com renamed MPPT_NODE
- net MPPT_NODE: now also Q7.3 (S), Q8.2 (D)
- net SOLR_IN_F: no longer names the net of F1.2
- net SOLR_IN_F: now also J16.1, J17.1 (Pin_1), J19.1 (Pin_1); no longer CP1.1
- net SOLR_IN_M renamed SOLR_MPPT_IN
- net SOLR_MPPT_IN: now also C22.2, CP1.1, CP2.1, U8.3 (IP-), U8.4 (IP-), U9.2 (SRC), U9.3 (IN); no longer C18.1
- net Solr_P renamed SOLR_RAW+
- net SOLR_RAW+: now also C17.2, D2.2 (A2), Q2.2 (D)
- new net: DZ1.1 (A), DZ1.3 (A), R20.1
- new net: C17.1, C18.1, D4.2 (A), Q1.3 (C), Q2.1 (G), Q3.1 (G), R18.2
- new net: C26.2, U10.18 (CAP)
- new net: C43.1, U14.21 (XOUT), Y2.1
- new net: C42.1, U14.20 (XIN), Y2.3
- new net: Q1.2 (E), R17.1
- new net: JP2.1 (A), Q4.2 (D), U9.8 (OUT)
- new net: D6.2 (A), R39.1
- new net: R28.2, U11.5 (LVG)
- new net: R27.2, U11.7 (HVG)
- new net: D5.2 (A), R21.1
- new net: Q1.1 (B), R19.2
- new net: J20.3 (Pin_3), R38.1
- new net: C39.1, C40.1, C41.1, U14.23 (DVDD), U14.45 (VREG_VOUT), U14.50 (DVDD)
- new net: J20.1 (Pin_1), R37.1
- new net: Q2.3 (S), Q3.3 (S), R18.1
- new net: D7.2 (A), R40.1
- new net A1V66: R24.2, R25.1, U10.4 (Ain1-), U10.5 (Ain2-), U10.8 (Ain3-), U10.9 (Ain4-)
- new net ADC_CLK: U10.17 (CLKIN)
- new net ADC_MISO: U10.15 (DOUT), U14.14 (GPIO11)
- new net ADC_MOSI: U10.16 (DIN), U14.15 (GPIO12)
- new net ADC_SCLK: U10.14 (SCLK), U14.13 (GPIO10)
- new net CurSnsFault_Load: U14.7 (GPIO5), U15.6 (~{FAULT})
- new net CurSnsFault_Solr: U14.6 (GPIO4), U8.6 (~{FAULT})
- new net D+: R36.2, U14.47 (USB_D+)
- new net D-: R35.2, U14.46 (USB_D-)
- new net ENable: U12.5 (LBK), U14.36 (GPIO24)
- new net GPIO26: U14.38 (GPIO26)
- new net GPIO27: U14.39 (GPIO27)
- new net GPIO28: U14.40 (GPIO28)
- new net GPIO29: U14.41 (GPIO29)
- new net GPLED1: D6.1 (K), U14.18 (GPIO15)
- new net GPLED2: D7.1 (K), U14.27 (GPIO16)
- new net MOD_ID1: U14.28 (GPIO17)
- new net MOD_ID2: U14.29 (GPIO18)
- new net MP3V3: C19.2, C23.2, C24.2, C27.2, C28.2, C30.2, C33.1, C34.1, C35.1, C36.1, C37.1, C38.1, R24.1, R31.2, R34.1, R39.2, R40.2, U10.1 (AVDD), U10.20 (DVDD), U12.3 (VCC), U13.8 (VDD), U14.1 (IOVDD), U14.10 (IOVDD), U14.22 (IOVDD), U14.33 (IOVDD), U14.42 (IOVDD), U14.43 (ADC_AVDD), U14.44 (VREG_VIN), U14.48 (USB_VDD), U14.49 (IOVDD), U15.8 (VCC), U8.8 (VCC)
- new net MPPT_OUT_F: C46.1, C47.1, F2.2, L2.2
- new net MP_ADC_CLK: TVS4.1 (A1)
- new net MP_BattPwr_P: D3.2 (A), D5.1 (K), DZ1.2 (K)
- new net MP_CAN_H: TVS1.1 (A1), U12.7 (CANH)
- new net MP_CAN_L: TVS1.2 (A2), U12.6 (CANL)
- new net MP_UART_RX: J21.2 (Pin_2), TVS3.1 (A1), U14.2 (GPIO0)
- new net MP_UART_TX: J21.3 (Pin_3), TVS3.2 (A2), U14.3 (GPIO1)
- new net ModeSel: U12.8 (Rs), U14.37 (GPIO25)
- new net QSPI_SCLK: U13.6 (SCK), U14.52 (QSPI_SCLK)
- new net QSPI_SD0: U13.5 (DI/IO0), U14.53 (QSPI_SD0)
- new net QSPI_SD1: U13.2 (DO/IO1), U14.55 (QSPI_SD1)
- new net QSPI_SD2: U13.3 (~{WP}/IO2), U14.54 (QSPI_SD2)
- new net QSPI_SD3: U13.7 (~{HOLD}/IO3), U14.51 (QSPI_SD3)
- new net RXD: U12.4 (R), U14.35 (GPIO23)
- new net SOLR_IV: JP1.2 (B), U8.1 (IP+), U8.2 (IP+)
- new net SOLR_LIM: C18.2, D4.1 (K), JP1.1 (A), Q3.2 (D), R21.2
- new net SWCLK: R37.2, U14.24 (SWCLK)
- new net SWDIO: R38.2, U14.25 (SWDIO)
- new net TXD: U12.1 (D), U14.34 (GPIO22)
- new net USB_D+: J22.3 (D+), R36.1
- new net USB_D-: J22.2 (D-), R35.1
- new net VCur_Load+: C32.2, U10.10 (Ain4+), U15.7 (VIOUT)
- new net VCur_Solr+: C21.2, U10.6 (Ain2+), U8.7 (VIOUT)
- new net ~{ADC_CS}: U10.12 (~{CS}), U14.16 (GPIO13)
- new net ~{ADC_DRDY}: U10.13 (~{DRDY}), U14.17 (GPIO14)
- new net ~{ALARM}: U14.30 (GPIO19)
- new net ~{MPPT_ALARM}: TVS4.2 (A2)
- new net ~{MPPT_RESET}: TVS2.2 (A2)
- new net ~{QSPI_CS}: R31.1, U13.1 (~{CS}), U14.56 (~{QSPI_CS})
- new net ~{RESET}: R34.2, SW2.2 (B), U14.26 (RUN)
- new net ~{SYNC}/~{RESET}: U10.11 (~{SYNC}/~{RESET}), U14.31 (GPIO20)
- no-connect marks 0 -> 8
Other:
- note added: "-"
- note added: "- +"
- note added: "- Pair of FETs act as bidir switch, preventing flow in and out of solr leads when switched off. - 470K Res is ?? unsure purpose. - Zener enables FETs to switch off if solr in has reverse polarity. - Bipolar Q enables MCU to actively dswitch off solr (rather than only reverse polarity events)"
- note added: "10"
- note added: "12MHz ABRACON"
- note added: "16V - 48V"
- note added: "18..24V Max 25A"
- note added: "22"
- note added: "33"
- note added: "42"
- note added: "43"
- note added: "48"
- note added: "49"
- note added: "50"
- note added: ">"
- note added: "ADC"
- note added: "AMASS XT30PW-M high-current dual pin connector, 30A. Mating plug XT30PW-F or similar."
- note added: "Because square wave current, the instantaneous current will be much higher max than the average."
- note added: "CONSOLE"
- note added: "CUI PJ-082BH high-current (10A) DC Barrel socket, centre positive. Nom 5.5mm/2.5mm (actual 6mm)"
- note added: "Cap current change will be large consider third cap here to share load. Panasonic TP series SMD/can Kemer PHA225 series axial 41x18mm"
- note added: "Current limit"
- note added: "Current->Voltage sensor & potential divider, linked to ADC/MCU to measure input I & V."
- note added: "Current->Voltage sensor & potential divider, linked to ADC/MCU to measure input I & V. Cap CP1 stores current while PWM has switched Q4 off, smoothing the load on the panels. CP2 helps manage higher frequency changes."
- note added: "I/V Sampling ADC"
- note added: "Ideal Diode"
- note added: "Load I-V Sense"
- note added: "Long term clip voltage"
- note added: "MPPT Controller"
- note added: "Max 25A & ~300W"
- note added: "Minimize track length"
- note added: "Minimize track length no vias"
- note added: "Power Filter"
- note added: "Prevent backfeed"
- note added: "Prevent power from flowing back into the power input (when Panel/Input Volts < Batt Volts)."
- note added: "RP2040 MCU in charge of ADC & PWM control."
- note added: "Reverse polarity, Input Switch"
- note added: "SWD Debug"
- note added: "SWDEBUG"
- note added: "Short term clip voltage"
- note added: "Simultaneous sampling 16/24 bit ADC, measures current and voltage as part of feedback control loop."
- note added: "Solar/Power Input & Fuse"
- note added: "Supplementary System Feed"
- note added: "These caps are on the MPPT side of the sensor so the sensor current is more stable as current flows in/out."
- note added: "To PSU: 30V Zener Limit, 40V TVS protection 1R,1W series resistor. Irmax = 30V/1R = 30A (short to gnd) ouch! PSU current expected is ~200..400mA. Design Imax out of PSU ~= 2A/12V = 24W (regulator spec). So for 1R, with 16V and 30V feed voltage: at 30V, 24W = (24/30) = 0.8A => Vr is 1R*0.8A = 0.8V, so Heat = 0.8*0.8 = 0.64W. at 16V, 24W = (24/16) = 1.5A => Vr is 1R*1.5A = 1.5V, so Heat = 1.5*1.5 =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"
- note added: "Vds < 100V Ids < 120A Qg ~ 150nC"
- note added: "Vds < 80V Ids < 147A Qg ~ 130nC"
- note added: "factor = 10/(10+470) = 0.0208"
- note added: "http://mail.components101.com/articles/design-guide-pmos-mosfet-for-reverse-voltage-polarity-protection"
- note added: "https://electronics.stackexchange.com/questions/35773/communication-between-multiple-microcontrollers#35776"
- note added: "https://github.com/KevinOConnor/can2040/"
- note added: "https://ibex.tech/resources/geek-area/electronics/mosfets/using-mosfets-as-general-switches"
- note added: "smoothing"
- note added: "|"
- note added: "≈0.35mA↓"
- note removed: "15V - 48V"
- note removed: "Load I-V Sense, PSU takeoff"
- note removed: "factor = 1 / (1+33) = 0.03"
- note removed: "~12V - ~18V"
- title: SolarPump v3 -> SolarPump v4
- moved on the sheet: C19, C20, C21, C22, C25, C31, CP1, CP3, HS1, HS2, L1, Q4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
