File: output.kicad_sch (KiCad schematic)
At the start: 40 parts, among them Q10 Si2306BDS, Q11 IRLB8721PBF, Q12 IRLB8721PBF, Q7 IRLB8721PBF, Q8 IRLB8721PBF, Q9 Si2306BDS, U11 L6398D, U12 ACS758xCB

Commit message: Further works...
Parts:
- removed D10, D9: B140-E3, Diode_SMD:D_SMA, symbol Device:D_Schottky
- removed HS4, HS5: HSink, MountingHole:MountingHole_2.7mm_M2.5_Pad_Via, symbol Mechanical:Heatsink_Pad
- removed Q10, Q9: Si2306BDS, Package_TO_SOT_SMD:SOT-23, symbol solarpump:Si2306BDS
- removed R37, R38, R39, R40: 10k, Resistor_SMD:R_0805_2012Metric_Pad1.20x1.40mm_HandSolder, symbol Device:R_Small
- removed U12: ACS758xCB, solarpump:Allegro_CB_PFF, symbol Sensor_Current:ACS758xCB-050B-PFF
- added C100, C103: 1uF, Capacitor_SMD:C_0603_1608Metric, symbol Device:C_Small
- added C101, C102, C91, C93, C94, C95, C96, C97, C98, C99: 0.1uF, Capacitor_SMD:C_0402_1005Metric, symbol Device:C_Small
- added C104, C105: 12pF, Capacitor_SMD:C_0402_1005Metric, symbol Device:C_Small
- added C79, C80, C81, C82, C87, C88: 0.1uF, Capacitor_SMD:C_0603_1608Metric, symbol Device:C_Small
- added D19, D22, D23: SMAJ54CA, Diode_SMD:D_SMA, symbol Diode:SMAJ54CA
- added D24, D25: Red,150mcd, LED_SMD:LED_1206_3216Metric_Pad1.42x1.75mm_HandSolder, symbol Device:LED
- added F3, F4: Fuse 25A, Fuse:Fuse_Schurter_UMZ250, symbol Device:Fuse
- added J26, J27: JST SM03B-SRSS-TB, Connector_JST:JST_SH_SM03B-SRSS-TB_1x03-1MP_P1.00mm_Horizontal, symbol Connector_Generic_MountingPin:Conn_01x03_MountingPin
- added J28: USB_B_Micro, Connector_USB:USB_Micro-B_Amphenol_10104110_Horizontal, symbol Connector:USB_B_Micro
- added J29: OP_Wire_Aux_P, Connector_Wire:SolderWire-2sqmm_1x01_D2mm_OD3.9mm, symbol Connector:Conn_01x01_Socket
- added J30: OP_Wire_Aux_N, Connector_Wire:SolderWire-2sqmm_1x01_D2mm_OD3.9mm, symbol Connector:Conn_01x01_Socket
- added J31: OP_Wire_Pump_P, Connector_Wire:SolderWire-2sqmm_1x01_D2mm_OD3.9mm, symbol Connector:Conn_01x01_Socket
- added J32: OP_Wire_Pump_N, Connector_Wire:SolderWire-2sqmm_1x01_D2mm_OD3.9mm, symbol Connector:Conn_01x01_Socket
- added J33, J34: Amass_XT30PW, solarpump:Amass_XT30PW, symbol solarpump:Amass_XT30PW
- added JP6: HIN_LIN, Jumper:SolderJumper-3_P1.3mm_Bridged2Bar12_RoundedPad1.0x1.5mm_NumberLabels, symbol Jumper:Jumper_3_Bridged12
- added Q12, Q13: IRLB8721PBF, Package_TO_SOT_THT:TO-220-3_Vertical, symbol Transistor_FET:IRLB8721PBF
- added R73: 33K,1%, Resistor_SMD:R_0603_1608Metric, symbol Device:R_Small
- added R74: 1K,1%, Resistor_SMD:R_0603_1608Metric, symbol Device:R_Small
- added R80, R81: 4.7k,0.5%, Resistor_SMD:R_0603_1608Metric, symbol Device:R_Small
- added R84, R89: 10K, Resistor_SMD:R_0603_1608Metric, symbol Device:R_Small
- added R90, R91: 27R, Resistor_SMD:R_0603_1608Metric, symbol Device:R_Small
- added R92, R93: 100R, Resistor_SMD:R_0603_1608Metric, symbol Device:R_Small
- added R94, R95: 72R, Resistor_SMD:R_0603_1608Metric, symbol Device:R_Small
- added SW9: SW_RESET, Button_Switch_SMD:SW_SPST_B3U-1000P, symbol Switch:SW_SPST
- added TVS10, TVS11, TVS8, TVS9: TVS, Package_TO_SOT_SMD:SOT-23, symbol Diode:PESD2IVN48T
- added U22, U26: ACS71240LLCBTR-025B3, Package_SO:SOIC-8_3.9x4.9mm_P1.27mm, symbol Sensor_Current:ACS71240LLCBTR-025B3
- added U24: ADS1115IDGS, Package_SO:TSSOP-10_3x3mm_P0.5mm, symbol Analog_ADC:ADS1115IDGS
- added U25: ADS131M04-PW, Package_SO:TSSOP-20_4.4x6.5mm_P0.65mm, symbol solarpump:ADS131M04-PW
- added U27: SN65HVD234, Package_SO:SOIC-8_3.9x4.9mm_P1.27mm, symbol Interface_CAN_LIN:SN65HVD233
- added U28: W25Q32JV, Package_SON:WSON-8-1EP_6x5mm_P1.27mm_EP3.4x4mm, symbol Memory_Flash_Extra:W25Q64JV
- added U29: 2EDN752x, Package_SO:Infineon_PG-DSO-8-43, symbol Driver_FET:2EDN752x
- added U30: RP2040, Package_DFN_QFN:QFN-56-1EP_7x7mm_P0.4mm_EP3.2x3.2mm_ThermalVias, symbol solarpump:RP2040
- added Y3: XYDBPCNANF-12MHZ, Crystal:Crystal_SMD_2520-4Pin_2.5x2.0mm, symbol Device:Crystal_GND24_Small
- C83: renamed from C39; value 2nF, 50V -> 2nF, 50V, Low ESR
- C84: renamed from C40; value 22uF,25V -> 22uF,>35V; footprint Capacitor_SMD:C_0805_2012Metric_Pad1.18x1.45mm_HandSolder -> Capacitor_Tantalum_SMD:CP_EIA-7360-38_Kemet-E
- C85: renamed from C41; value 22uF,25V -> 22uF,>35V; footprint Capacitor_SMD:C_0805_2012Metric_Pad1.18x1.45mm_HandSolder -> Capacitor_Tantalum_SMD:CP_EIA-7360-38_Kemet-E
- C86: renamed from C42; value 22uF,25V -> 22uF,>35V; footprint Capacitor_SMD:C_0805_2012Metric_Pad1.18x1.45mm_HandSolder -> Capacitor_Tantalum_SMD:CP_EIA-7360-38_Kemet-E
- C89: renamed from C43; footprint Capacitor_SMD:C_0805_2012Metric_Pad1.18x1.45mm_HandSolder -> Capacitor_SMD:C_0603_1608Metric
- C90: renamed from C44; footprint Capacitor_SMD:C_0805_2012Metric_Pad1.18x1.45mm_HandSolder -> Capacitor_SMD:C_0402_1005Metric
- C92: renamed from C45; footprint Capacitor_SMD:C_0805_2012Metric_Pad1.18x1.45mm_HandSolder -> Capacitor_SMD:C_0402_1005Metric
- CP7: value 470uF,25V -> 470uF,50V
- L5: value 68uH -> 68uH,15A
- R75: renamed from R30; footprint Resistor_SMD:R_0805_2012Metric_Pad1.20x1.40mm_HandSolder -> Resistor_SMD:R_0603_1608Metric
- R76: renamed from R31; footprint Resistor_SMD:R_0805_2012Metric_Pad1.20x1.40mm_HandSolder -> Resistor_SMD:R_0603_1608Metric
- R77: renamed from R32; footprint Resistor_SMD:R_0805_2012Metric_Pad1.20x1.40mm_HandSolder -> Resistor_SMD:R_0603_1608Metric
- R78: renamed from R33; footprint Resistor_SMD:R_0805_2012Metric_Pad1.20x1.40mm_HandSolder -> Resistor_SMD:R_0603_1608Metric
- R79: renamed from R34; footprint Resistor_SMD:R_0805_2012Metric_Pad1.20x1.40mm_HandSolder -> Resistor_SMD:R_0603_1608Metric
- R82: renamed from R35; footprint Resistor_SMD:R_0805_2012Metric_Pad1.20x1.40mm_HandSolder -> Resistor_SMD:R_0603_1608Metric
- R83: renamed from R36; value 1k -> 1K,1%; footprint Resistor_SMD:R_0805_2012Metric_Pad1.20x1.40mm_HandSolder -> Resistor_SMD:R_0603_1608Metric
- R85: renamed from R41; footprint Resistor_SMD:R_0805_2012Metric_Pad1.20x1.40mm_HandSolder -> Resistor_SMD:R_0603_1608Metric
- R86: renamed from R42; footprint Resistor_SMD:R_0805_2012Metric_Pad1.20x1.40mm_HandSolder -> Resistor_SMD:R_0603_1608Metric
- R87: renamed from R43; footprint Resistor_SMD:R_0805_2012Metric_Pad1.20x1.40mm_HandSolder -> Resistor_SMD:R_0603_1608Metric
- R88: renamed from R44; footprint Resistor_SMD:R_0805_2012Metric_Pad1.20x1.40mm_HandSolder -> Resistor_SMD:R_0603_1608Metric
- renumbered D11 to D20, D12 to D21, HS6 to HS3, HS7 to HS4, Q7 to Q10, Q8 to Q11, Q11 to Q14, Q12 to Q15, U11 to U23
Connections:
- net GNDA is gone; now on net OPGND: C90.2
- net VOutput+: now also U24.6 (AIN2), U25.7 (Ain3+)
- net OP_LC: now reaches C84.1, C85.1, C86.1, CP7.1, L5.2
- net OP_LC: now also U26.3 (IP-), U26.4 (IP-)
- net at Q10.1 (G), R76.1, R78.1: now also Q12.1 (G)
- net at Q11.1 (G), R77.1, R79.1: now also Q13.1 (G)
- net OP_Pmp_G: now reaches Q14.1 (G), R85.1, R87.2
- net at R85.2: now also U29.7 (OUTA)
- net at R86.2: now also U29.5 (OUTB)
- net OP_Aux_G: now reaches Q15.1 (G), R86.1, R88.1
- net +12V renamed OP12V
- net OP12V: now also U29.6 (VDD)
- net +3V3 renamed OP3V3
- net OP3V3: now also C100.1, C81.1, C82.2, C87.2, C88.2, C93.2, C94.2, C95.1, C96.1, C97.1, C98.1, C99.1, R80.1, R84.2, R89.1, R94.2, R95.2, U22.8 (VCC), U24.8 (VDD), U25.1 (AVDD), U25.20 (DVDD), U26.8 (VCC), U27.3 (VCC), U28.8 (VDD), U30.1 (IOVDD), U30.10 (IOVDD), U30.22 (IOVDD), U30.33 (IOVDD), U30.42 (IOVDD), U30.43 (ADC_AVDD), U30.44 (VREG_VIN), U30.48 (USB_VDD), U30.49 (IOVDD)
- net BUCK_PWMhi renamed OP_BUCK_PWMhi
- net OP_BUCK_PWMhi: now also JP6.3 (B), U30.11 (GPIO8)
- net BUCK_PWMlo: no longer names the net of U23.3 (~{LIN})
- net BUCK_PWMlo: now also JP6.2 (C)
- net GND renamed OPGND
- net OPGND: now also C100.2, C101.2, C102.2, C103.2, C104.2, C105.2, C79.2, C80.2, C81.2, C82.1, C87.1, C88.1, C91.1, C93.1, C94.1, C95.2, C96.2, C97.2, C98.2, C99.2, D19.1 (A1), J26.2 (Pin_2), J26.MP (MountPin), J27.1 (Pin_1), J27.MP (MountPin), J28.5 (GND), J28.6 (Shield), J33.MP (MountPin), J34.MP (MountPin), Q13.3 (S), R74.2, R81.2, SW9.1 (A), TVS10.3 (common), TVS11.3 (common), TVS8.3 (common), TVS9.3 (common), U22.5 (GND), U24.1 (ADDR), U24.3 (GND), U25.19 (DGND), U25.2 (AGND), U26.5 (GND), U27.2 (GND), U28.4 (GND), U28.9 (GND), U29.3 (GND), U29.9 (EP), U30.19 (TESTEN), U30.57 (GND), Y3.2, Y3.4
- net Load_P renamed OP_MainInput
- net OP_MainInput: now also Q12.2 (D), R73.1, U22.1 (IP+), U22.2 (IP+)
- net OUT_Com renamed BUCK_NODE
- net BUCK_NODE: now also Q12.3 (S), Q13.2 (D)
- net OUT_Hvg renamed OP_Hvg
- net OUT_Lvg renamed OP_Lvg
- removed net Out_Aux+: D20.1 (K), D21.1 (K), R82.1
- net Out_Aux- renamed OP_Aux_N
- net OP_Aux_N: now also D23.1 (A1), J30.1 (Pin_1), J34.2 (Pin_2)
- net Out_Pump- renamed OP_Pmp_N
- net OP_Pmp_N: now also D22.1 (A1), J32.1 (Pin_1), J33.2 (Pin_2)
- net VCurrent_Output+ renamed VCur_Output+
- net VCur_Output+: now also U24.7 (AIN3), U25.10 (Ain4+), U26.7 (VIOUT)
- new net: D20.1 (K), D22.2 (A2), F3.1, J31.1 (Pin_1), J33.1 (Pin_1)
- new net: D21.1 (K), D23.2 (A2), F4.1, J29.1 (Pin_1), J34.1 (Pin_1)
- new net: J26.1 (Pin_1), R92.1
- new net: J26.3 (Pin_3), R93.1
- new net: C101.1, C102.1, C103.1, U30.23 (DVDD), U30.45 (VREG_VOUT), U30.50 (DVDD)
- new net: C105.1, U30.21 (XOUT), Y3.1
- new net: C104.1, U30.20 (XIN), Y3.3
- new net: D25.2 (A), R95.1
- new net: C91.2, U25.18 (CAP)
- new net: D24.2 (A), R94.1
- new net A1V66: R80.2, R81.1, U25.4 (Ain1-), U25.5 (Ain2-), U25.8 (Ain3-), U25.9 (Ain4-)
- new net ADC_CLK: TVS9.1 (A1), U25.17 (CLKIN)
- new net ADC_MISO: U25.15 (DOUT), U30.14 (GPIO11)
- new net ADC_MOSI: U25.16 (DIN), U30.15 (GPIO12)
- new net ADC_SCLK: U25.14 (SCLK), U30.13 (GPIO10)
- new net CAN_H: TVS11.1 (A1), U27.6 (CANL)
- new net CAN_L: TVS11.2 (A2), U27.7 (CANH)
- new net D+: R91.2, U30.47 (USB_D+)
- new net D-: R90.2, U30.46 (USB_D-)
- new net ENable: U27.5 (LBK), U30.36 (GPIO24)
- new net GPIO26: U30.38 (GPIO26)
- new net GPIO27: U30.39 (GPIO27)
- new net GPIO28: U30.40 (GPIO28)
- new net GPIO29: U30.41 (GPIO29)
- new net GPLED1: D24.1 (K), U30.18 (GPIO15)
- new net GPLED2: D25.1 (K), U30.27 (GPIO16)
- new net InputCurSns_Fault: U22.6 (~{FAULT})
- new net Input_CurSnsFault: U30.8 (GPIO6)
- new net MOD_ID1: U30.28 (GPIO17)
- new net MOD_ID2: U30.29 (GPIO18)
- new net ModeSel: U27.8 (Rs), U30.37 (GPIO25)
- new net OP5V: J28.1 (VBUS)
- new net OP_BUCK_PWMlo: JP6.1 (A), U30.12 (GPIO9)
- new net OP_Enable_Aux: U29.4 (INB)
- new net OP_Enable_Pmp: U29.2 (INA), U30.7 (GPIO5)
- new net OP_I2C.SCL: U24.9 (SDA), U30.5 (GPIO3)
- new net OP_I2C.SDA: U24.10 (SCL), U30.4 (GPIO2)
- new net OP_I2C.~{IRQ}: U24.2 (ALERT/RDY), U30.6 (GPIO4)
- new net OP_Load_P: D19.2 (A2), U22.3 (IP-), U22.4 (IP-)
- new net OP_MainOutput: F3.2, F4.2, R82.1, U26.1 (IP+), U26.2 (IP+)
- new net OP_UART_RX: J27.2 (Pin_2), U30.2 (GPIO0)
- new net OP_UART_TX: J27.3 (Pin_3), U30.3 (GPIO1)
- new net OutputCurSns_Fault: U26.6 (~{FAULT})
- new net Output_CurSnsFault: U30.9 (GPIO7)
- new net QSPI_SCLK: U28.6 (SCK), U30.52 (QSPI_SCLK)
- new net QSPI_SD0: U28.5 (DI/IO0), U30.53 (QSPI_SD0)
- new net QSPI_SD1: U28.2 (DO/IO1), U30.55 (QSPI_SD1)
- new net QSPI_SD2: U28.3 (~{WP}/IO2), U30.54 (QSPI_SD2)
- new net QSPI_SD3: U28.7 (~{HOLD}/IO3), U30.51 (QSPI_SD3)
- new net RXD: U27.4 (R), U30.35 (GPIO23)
- new net SWCLK: R92.2, U30.24 (SWCLK)
- new net SWDIO: R93.2, U30.25 (SWDIO)
- new net TXD: U27.1 (D), U30.34 (GPIO22)
- new net UART_RX: TVS10.1 (A1)
- new net UART_TX: TVS10.2 (A2)
- new net USB_D+: J28.3 (D+), R91.1
- new net USB_D-: J28.2 (D-), R90.1
- new net VCur_Input+: C79.1, U22.7 (VIOUT), U24.5 (AIN1), U25.6 (Ain2+)
- new net VInput+: C80.1, R73.2, R74.1, U24.4 (AIN0), U25.3 (Ain1+)
- new net ~{ADC_CS}: U25.12 (~{CS}), U30.16 (GPIO13)
- new net ~{ADC_DRDY}: U25.13 (~{DRDY}), U30.17 (GPIO14)
- new net ~{ALARM}: TVS8.2 (A2), U30.30 (GPIO19)
- new net ~{QSPI_CS}: R84.1, U28.1 (~{CS}), U30.56 (~{QSPI_CS})
- new net ~{RESET}: R89.2, SW9.2 (B), TVS9.2 (A2), U30.26 (RUN)
- new net ~{SYNC}/~{RESET}: U25.11 (~{SYNC}/~{RESET}), U30.31 (GPIO20)
- no-connect marks 0 -> 5
Other:
- note added: "10"
- note added: "12MHz ABRACON"
- note added: "22"
- note added: "33"
- note added: "42"
- note added: "43"
- note added: "48"
- note added: "49"
- note added: "50"
- note added: "ADC"
- note added: "BUCK Output Controller"
- note added: "CONSOLE"
- note added: "Has Int 400kR to vdd Ext pull high 10kR?"
- note added: "I/V Sampling ADC"
- note added: "Input I-V Sense"
- note added: "Minimise gap btw cap and IC."
- note added: "Minimize track length"
- note added: "Option: Dup FETS in parallel?"
- note added: "RP2040 MCU in charge of ADC & PWM control."
- note added: "SWD Debug"
- note added: "SWDEBUG"
- note added: "Simultaneous sampling 16/24 bit ADC, measures current and voltage as part of feedback control loop."
- note added: "≈0.35mA↓"
- title: SolarPump v3 -> SolarPump v4
- moved on the sheet: C83, C84, C85, C86, C89, C90, C92, CP7, D20, D21, HS3, HS4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
