File: psu.kicad_sch (KiCad schematic)
At the start: 30 parts, among them U7 LM2593HVS-ADJ, U8 LM2575S-5, U9 LM2575S-3.3

Commit message: Schematic + pcb 1.3.3
Parts:
- added C59: 47uF, Capacitor_SMD:C_1206_3216Metric_Pad1.33x1.80mm_HandSolder, symbol Device:C_Small
- added D19: Red,150mcd, LED_SMD:LED_1206_3216Metric_Pad1.42x1.75mm_HandSolder, symbol Device:LED
- added D20, D21: Orange,160mcd, LED_SMD:LED_1206_3216Metric_Pad1.42x1.75mm_HandSolder, symbol Device:LED
- added R58: 620R, Resistor_SMD:R_0805_2012Metric_Pad1.20x1.40mm_HandSolder, symbol Device:R_Small
- added R59, R61: 160R, Resistor_SMD:R_0805_2012Metric_Pad1.20x1.40mm_HandSolder, symbol Device:R_Small
- C33: value 4.7uF,25V -> 4.7uF,16V
- CP4: value 470uF, 25V -> 470uF,25V
- CP5, CP6: value 390uF, 10V -> 390uF,10V
- D13: value PLZ3V6A, 3.45-3.7V -> PLZ3V6A,3.45-3.7V
Connections:
- net +12V: now also R58.1
- net +3V3: now also R61.1
- net +5V: now also C59.1, R59.1
- net GND: now also C59.2, D19.1 (K), D20.1 (K), D21.1 (K)
- new net: D21.2 (A), R61.2
- new net: D19.2 (A), R58.2
- new net: D20.2 (A), R59.2
Other:
- note added: "3.3V, 1A switch reg. (ADC/Logic)"
- note added: "Consider ADP122AUJZ-3.3-R7: 300mA 3.3V LDO in TSOT-23-5, MaxV 5.5V, quiescent 45uA or ADP3333ARMZ3.3R7: 300mA 3.3V LDO in MSOP-8, MaxV 12V, quiescent 75uA"
- note added: "Consider LV2862: 600mA 5V o/p in SOT23-6 pkg. L=22uH"
- note removed: "3.3V, 1A switch reg. (MCU)"
- moved on the sheet: C25, C26, C27, C28, C29, C30, C31, C32, C33, C34, C49, C50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

Commit message: Further works...
Parts:
- removed C30, C31: 47uF, Capacitor_THT:CP_Radial_D6.3mm_P2.50mm, symbol Device:C_Small
- removed C32: 4.7uF,25V, Capacitor_SMD:C_0805_2012Metric_Pad1.18x1.45mm_HandSolder, symbol Device:C_Small
- removed C33: 4.7uF,16V, Capacitor_SMD:C_0805_2012Metric_Pad1.18x1.45mm_HandSolder, symbol Device:C_Small
- removed C34, C59: 47uF, Capacitor_SMD:C_1206_3216Metric_Pad1.33x1.80mm_HandSolder, symbol Device:C_Small
- removed CP5, CP6: 390uF,10V, Capacitor_THT:CP_Radial_D8.0mm_P3.50mm, symbol Device:C_Polarized_Small
- removed D20, D21: Orange,160mcd, LED_SMD:LED_1206_3216Metric_Pad1.42x1.75mm_HandSolder, symbol Device:LED
- removed D7, D8: B140-E3, Diode_SMD:D_SMA, symbol Device:D_Schottky
- removed L3: 100uH, Inductor_SMD:L_10.4x10.4_H4.8, symbol Device:L_Ferrite
- removed R59, R61: 160R, Resistor_SMD:R_0805_2012Metric_Pad1.20x1.40mm_HandSolder, symbol Device:R_Small
- removed U8: LM2575S-5, solarpump:TO-263-5_TabPin3, symbol Regulator_Switching:LM2576S-5
- removed U9: LM2575S-3.3, solarpump:TO-263-5_TabPin3, symbol Regulator_Switching:LM2576S-3.3
- added BT1: Li-Ion 3V7, Connector_JST:JST_PH_B2B-PH-K_1x02_P2.00mm_Vertical, symbol Device:Battery_Cell
- added C55: 10uF,25V, Capacitor_SMD:C_0805_2012Metric_Pad1.18x1.45mm_HandSolder, symbol Device:C_Small
- added C56: 2.2uF,25V, Capacitor_SMD:C_0805_2012Metric_Pad1.18x1.45mm_HandSolder, symbol Device:C_Small
- added C57, C64: 0.1uF, Capacitor_SMD:C_0603_1608Metric, symbol Device:C_Small
- added C58: 4.7uF,16V Tant, Capacitor_SMD:C_0805_2012Metric_Pad1.18x1.45mm_HandSolder, symbol Device:C_Polarized_Small
- added C59: 1uF,16V Tant, Capacitor_SMD:C_0805_2012Metric_Pad1.18x1.45mm_HandSolder, symbol Device:C_Polarized_Small
- added C60: 4.7uF, Capacitor_SMD:C_0603_1608Metric, symbol Device:C_Small
- added C62: 2.2uF,10V, Capacitor_SMD:C_0805_2012Metric_Pad1.18x1.45mm_HandSolder, symbol Device:C_Small
- added C63: 4.7uF,10V, Capacitor_SMD:C_0805_2012Metric_Pad1.18x1.45mm_HandSolder, symbol Device:C_Small
- added D11: B150-E3,50V, Diode_SMD:D_SMA, symbol Device:D_Schottky
- added D12, D13: LED_CHR, LED_SMD:LED_0603_1608Metric, symbol Device:LED_Small
- added D14: Orange,160mcd, LED_SMD:LED_1206_3216Metric_Pad1.42x1.75mm_HandSolder, symbol Device:LED
- added R45: 100K, Resistor_SMD:R_0603_1608Metric, symbol Device:R_Small
- added R46: 54.9K,0.5%, Resistor_SMD:R_0603_1608Metric, symbol Device:R_Small
- added R47: 10K,0.5%, Resistor_SMD:R_0603_1608Metric, symbol Device:R_Small
- added R48: 2K, Resistor_SMD:R_0603_1608Metric, symbol Device:R_Small
- added R49: 25K, Resistor_SMD:R_0603_1608Metric, symbol Device:R_Small
- added R50, R51: 680R, Resistor_SMD:R_0603_1608Metric, symbol Device:R_Small
- added R52: 220R, Resistor_SMD:R_0603_1608Metric, symbol Device:R_Small
- added TH3: 10K NTC, solarpump:SolderWire-0.15sqmm_1x02_P3.5mm_D0.5mm_OD1.5mm, symbol Device:Thermistor_NTC
- added U17: LV2862XDDC, Package_TO_SOT_SMD:SOT-23-6, symbol Regulator_Switching:LV2862XDDC
- added U18: MCP73871-2CC, Package_DFN_QFN:QFN-20-1EP_4x4mm_P0.5mm_EP2.5x2.5mm, symbol Battery_Management:MCP73871-2CC
- added U19: AP7361C-33ER-13, Package_TO_SOT_SMD:SOT-223-3_TabPin2, symbol Regulator_Linear:AP7361C-33E
- added U20: LM809-M3X 3.08, Package_TO_SOT_SMD:SOT-23, symbol Power_Supervisor:LM809
- C49: renamed from C26; footprint Capacitor_SMD:C_0805_2012Metric_Pad1.18x1.45mm_HandSolder -> Capacitor_SMD:C_0603_1608Metric
- C50: renamed from C27; footprint Capacitor_SMD:C_0805_2012Metric_Pad1.18x1.45mm_HandSolder -> Capacitor_SMD:C_0603_1608Metric
- C51: renamed from C50; footprint Capacitor_SMD:C_0805_2012Metric_Pad1.18x1.45mm_HandSolder -> Capacitor_SMD:C_0603_1608Metric; DNF DNF -> (none)
- C52: renamed from C28; footprint Capacitor_SMD:C_0805_2012Metric_Pad1.18x1.45mm_HandSolder -> Capacitor_SMD:C_0603_1608Metric
- C54: renamed from C49; footprint Capacitor_SMD:C_0805_2012Metric_Pad1.18x1.45mm_HandSolder -> Capacitor_SMD:C_0603_1608Metric; DNF DNF -> (none)
- D8: renamed from D6; value B140-E3 -> B150-E3,50V; DNF DNF -> (none)
- D9: renamed from D13; DNF DNF -> (none)
- L4: value 100uH -> 22uH, 750mA
- R41: renamed from R21; footprint Resistor_SMD:R_0805_2012Metric_Pad1.20x1.40mm_HandSolder -> Resistor_SMD:R_0603_1608Metric
- R42: renamed from R22; footprint Resistor_SMD:R_0805_2012Metric_Pad1.20x1.40mm_HandSolder -> Resistor_SMD:R_0603_1608Metric
- R43: renamed from R20; footprint Resistor_SMD:R_0805_2012Metric_Pad1.20x1.40mm_HandSolder -> Resistor_SMD:R_0603_1608Metric
- R44: renamed from R58; footprint Resistor_SMD:R_0805_2012Metric_Pad1.20x1.40mm_HandSolder -> Resistor_SMD:R_0603_1608Metric
- renumbered C25 to C48, C29 to C53, CP3 to CP4, CP8 to CP5, CP4 to CP6, D19 to D10, L2 to L3, U7 to U16
Connections:
- net +3V3: now also C63.1, C64.1, R52.1, U19.3 (VO), U20.3 (VCC); no longer L4.2
- net GND: now also BT1.2 (-), C55.2, C56.2, C58.2, C59.2, C60.1, C62.2, C63.2, C64.2, D11.2 (A), D14.1 (K), R47.2, R48.1, R49.1, TH3.2, U17.2 (GND), U18.10 (V_{SS}), U18.11 (V_{SS}), U18.21 (V_{SS}), U19.2 (GND), U20.1 (GND)
- net 5Vnode: now reaches L4.1
- net 5Vnode: now also C57.2, D11.1 (K), R46.1, U17.6 (SW)
- net 12Vnode: now reaches D8.1 (K), L3.1, U16.2 (OUT)
- net +12V renamed 12V
- net 12V: now also C55.1, C56.1, R45.1, U17.5 (VIN)
- net ~{REG_ERR} renamed ~{PSU_REG_ERR}
- new net: TH3.1, U18.5 (THERM)
- new net: BT1.1 (+), C60.2, U18.14 (V_{BAT}), U18.15 (V_{BAT}), U18.16 (V_{BAT_SENSE})
- new net: R49.2, U18.12 (PROG3)
- new net: R48.2, U18.13 (PROG1)
- new net: D13.1 (K), U18.6 (~{PG})
- new net: D12.1 (K), U18.8 (STAT1/~{LBO})
- new net: D12.2 (A), R50.2
- new net: D14.2 (A), R52.2
- new net: D13.2 (A), R51.2
- new net 5V: C62.1, R50.1, R51.1, U18.1 (OUT), U18.20 (OUT), U19.1 (VI)
- new net 5Vreg: C58.1, C59.1, L4.2, U18.17 (CE), U18.18 (IN), U18.19 (IN), U18.2 (VPCC), U18.3 (SEL)
- new net BPassC: C57.1, U17.1 (CB)
- new net FBack: R46.2, R47.1, U17.3 (FB)
- new net Shdwn: R45.2, U17.4 (~{SHDN})
- new net ~{PSU_RESET}: U20.2 (~{RESET})
- no-connect marks 0 -> 3
Other:
- note added: "12V"
- note added: "12V SMPS"
- note added: "3V3"
- note added: "3V3 LDO"
- note added: "5V"
- note added: "5V BOOST when run from Battery. Low Bat cutoff?"
- note added: "5V SMPS"
- note added: "5V/BAT"
- note added: "60V abs max input"
- note added: ">16V"
- note added: "BATTERY CHARGE/BACKUP"
- note added: "PWR-ON-RESET"
- note added: "SEL tied HIGH -> use 1.65/max 1.8A charge (otherwise USB) PROG1 => current limit. 2K sets 500mA PROG2 N/C because SEL is not USB PROG3 sets end of charge point. CE = charge enable, high to use Bat. THERM regulates Bat temp."
- note removed: "3.3V, 1A switch reg. (ADC/Logic)"
- note removed: "5V, 1A switch reg. (MCU/USB)"
- note removed: "Consider ADP122AUJZ-3.3-R7: 300mA 3.3V LDO in TSOT-23-5, MaxV 5.5V, quiescent 45uA or ADP3333ARMZ3.3R7: 300mA 3.3V LDO in MSOP-8, MaxV 12V, quiescent 75uA"
- note removed: "Consider LV2862: 600mA 5V o/p in SOT23-6 pkg. L=22uH"
- title: SolarPump v3 -> SolarPump v4
- moved on the sheet: C48, C49, C50, C51, C52, C53, C54, CP4, CP5, CP6, D10, D8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
